File: 6502/6502/6502.kicad_pcb (KiCad board)
At the start: 2 copper layers, 54 parts, among them J1 Jack-DC, J10 Conn_01x05, J11 DIN-6, J2 Conn_01x08, J3 Conn_01x08, J4 Conn_01x08, J5 Conn_01x16, J6 Conn_01x08, J7 Conn_01x08, J8 Conn_01x16, J9 Conn_01x06, SW1 SW_Push, U1 65C22S, U10 74LS08, U11 74HC14, U12 74HC595, U13 74HC595, U2 65C22S, U3 65C02S, U4 28C256, U5 65C51N, U6 62256, U7 PAL24, U8 NHD-0420H1Z, U9 74LS154, X1 ACO-4MHz, Y1 1.8432MHz

Commit message: changes
Connections:
- U11 pad 5: (no net) -> PS2_CLK
- U11 pad 6: (no net) -> Net-(U11-Pad6)
- U12 pad 11: Net-(D3-Pad2) -> Net-(U11-Pad6)
- U13 pad 11: Net-(D3-Pad2) -> Net-(U11-Pad6)
