File: 6502/6502/6502.sch (KiCad schematic (older format))
At the start: 1 part

Commit message: started schematic
Parts:
- removed U?: 74LS154, symbol 74xx:74LS154
- added C1, C10, C11, C12, C2, C3, C4, C5, C6, C7, C8, C9: 0.1uF, symbol Device:C
- added C13: 30pF, symbol Device:C
- added R1: 1K, symbol Device:R
- added R2: 1M, symbol Device:R
- added RV1: R_POT, symbol Device:R_POT
- added SW1: SW_Push, symbol Switch:SW_Push
- added U1, U2: 65C22S, Package_DIP:DIP-40_W15.24mm_Socket, symbol 6502:65C22S
- added U3: 65C02S, Package_DIP:DIP-40_W15.24mm_Socket, symbol 6502:65C02S
- added U4: 28C256, Package_DIP:DIP-28_W15.24mm_Socket, symbol 6502:28C256
- added U5: 65C51N, Package_DIP:DIP-28_W15.24mm_Socket, symbol 6502:65C51N
- added U6: 62256, Package_DIP:DIP-28_W15.24mm_Socket, symbol 6502:62256
- added U7: PAL24, symbol Logic_Programmable:PAL24
- added U8: NHD-0420H1Z, Display:NHD-0420H1Z, symbol Display_Character:NHD-0420H1Z
- added U9: 74LS154, symbol 74xx:74LS154
- added X1: ACO-xxxMHz, Oscillator:Oscillator_DIP-14, symbol Oscillator:ACO-xxxMHz
- added Y1: Crystal, symbol Device:Crystal
Connections:
- new net: U5.11 (~DTR), U5.16 (~DCD), U5.17 (~DSR)
- new net: C13.1, R2.1, U5.6 (XTLI), Y1.1
- new net: R2.2, U5.7 (XTLO), Y1.2
- new net: RV1.3, U8.2 (VDD)
- new net: RV1.2, U8.3 (VO)
- new net +5V: C1.2, C10.2, C11.2, C12.2, C2.2, C3.2, C4.2, C5.2, C6.2, C7.2, C8.2, C9.2, R1.1, U1.20 (VDD), U1.24 (CS1), U2.20 (VDD), U2.24 (CS1), U3.2 (RDY), U3.36 (BE), U3.38 (~SO), U3.6 (~NMI), U3.8 (VCC), U4.28 (VCC), U5.15 (VDD), U5.2 (CS0), U6.28 (VCC), U7.24 (VCC), U8.15 (A), U9.24 (VCC), X1.14 (Vcc)
- new net 1pa0: U2.2 (PA0)
- new net 1pa1: U2.3 (PA1)
- new net 1pa2: U2.4 (PA2)
- new net 1pa3: U2.5 (PA3)
- new net 1pa4: U2.6 (PA4)
- new net 1pa5: U2.7 (PA5)
- new net 1pa6: U2.8 (PA6)
- new net 1pa7: U2.9 (PA7)
- new net 1pb0: U2.10 (PB0)
- new net 1pb1: U2.11 (PB1)
- new net 1pb2: U2.12 (PB2)
- new net 1pb3: U2.13 (PB3)
- new net 1pb4: U2.14 (PB4)
- new net 1pb5: U2.15 (PB5)
- new net 1pb6: U2.16 (PB6)
- new net 1pb7: U2.17 (PB7)
- new net 2pa0: U1.2 (PA0)
- new net 2pa1: U1.3 (PA1)
- new net 2pa2: U1.4 (PA2)
- new net 2pa3: U1.5 (PA3)
- new net 2pa4: U1.6 (PA4)
- new net 2pa5: U1.7 (PA5)
- new net 2pa6: U1.8 (PA6)
- new net 2pa7: U1.9 (PA7)
- new net 2pb0: U1.10 (PB0)
- new net 2pb1: U1.11 (PB1)
- new net 2pb2: U1.12 (PB2)
- new net 2pb3: U1.13 (PB3)
- new net 2pb4: U1.14 (PB4)
- new net 2pb5: U1.15 (PB5)
- new net 2pb6: U1.16 (PB6)
- new net 2pb7: U1.17 (PB7)
- new net ACIA_CS: U5.3 (~CS1), U9.3 (S2)
- new net DEVICE_CS: U7.18 (NC/O0), U9.19 (E1)
- new net GND: C1.1, C10.1, C11.1, C12.1, C13.2, C2.1, C3.1, C4.1, C5.1, C6.1, C7.1, C8.1, C9.1, RV1.1, SW1.2, U1.1 (VSS), U2.1 (VSS), U3.21 (GND), U4.14 (GND), U5.1 (VSS), U6.14 (GND), U7.12 (GND), U8.1 (VSS), U8.16 (K), U9.12 (GND), X1.7 (GND)
- new net OE: U4.22 (~OE), U6.22 (~OE), U7.14 (LR/O4)
- new net PHI2: U1.25 (PHI2), U2.25 (PHI2), U3.37 (PHI2), U5.27 (PHI2), U7.1 (OD/CLK), X1.8 (OUT)
- new net RAM_CS: U6.20 (~CE), U7.16 (A1/O2)
- new net RESET: R1.2, SW1.1, U1.34 (~RES), U2.34 (~RES), U3.40 (~RESET), U5.4 (~RES)
- new net ROM_CS: U4.20 (~CE), U7.17 (A2/O1)
- new net RW: U1.22 (R~W), U2.22 (R~W), U3.34 (R/~W), U5.28 (R~W), U7.2 (I0)
- new net VIA1_CS: U2.23 (~CS2), U9.1 (S0)
- new net VIA2_CS: U1.23 (~CS2), U9.2 (S1)
- new net WE: U4.27 (~WE), U6.27 (~WE), U7.15 (A0/O3)
- new net a0: U1.38 (RS0), U2.38 (RS0), U3.9 (A0), U4.10 (A0), U5.13 (RS0), U6.10 (A0), U9.23 (A0)
- new net a1: U1.37 (RS1), U2.37 (RS1), U3.10 (A1), U4.9 (A1), U5.14 (RS1), U6.9 (A1), U9.22 (A1)
- new net a10: U3.19 (A10), U4.21 (A10), U6.21 (A10), U7.8 (I6)
- new net a11: U3.20 (A11), U4.23 (A11), U6.23 (A11), U7.7 (I5)
- new net a12: U3.22 (A12), U4.2 (A12), U6.2 (A12), U7.6 (I4)
- new net a13: U3.23 (A13), U4.26 (A13), U6.26 (A13), U7.5 (I3)
- new net a14: U3.24 (A14), U4.1 (A14), U6.1 (A14), U7.4 (I2)
- new net a15: U3.25 (A15), U7.3 (I1), U9.18 (E0)
- new net a2: U1.36 (RS2), U2.36 (RS2), U3.11 (A2), U4.8 (A2), U6.8 (A2), U9.21 (A2)
- new net a3: U1.35 (RS3), U2.35 (RS3), U3.12 (A3), U4.7 (A3), U6.7 (A3), U9.20 (A3)
- new net a4: U3.13 (A4), U4.6 (A4), U6.6 (A4)
- new net a5: U3.14 (A5), U4.5 (A5), U6.5 (A5)
- new net a6: U3.15 (A6), U4.4 (A6), U6.4 (A6)
- new net a7: U3.16 (A7), U4.3 (A7), U6.3 (A7)
- new net a8: U3.17 (A8), U4.25 (A8), U6.25 (A8), U7.10 (I8)
- new net a9: U3.18 (A9), U4.24 (A9), U6.24 (A9), U7.9 (I7)
- new net d0: U1.33 (D0), U2.33 (D0), U3.33 (D0), U4.11 (D0), U5.18 (D0), U6.11 (D0)
- new net d1: U1.32 (D1), U2.32 (D1), U3.32 (D1), U4.12 (D1), U5.19 (D1), U6.12 (D1)
- new net d2: U1.31 (D2), U2.31 (D2), U3.31 (D2), U4.13 (D2), U5.20 (D2), U6.13 (D2)
- new net d3: U1.30 (D3), U2.30 (D3), U3.30 (D3), U4.15 (D3), U5.21 (D3), U6.15 (D3)
- new net d4: U1.29 (D4), U2.29 (D4), U3.29 (D4), U4.16 (D4), U5.22 (D4), U6.16 (D4)
- new net d5: U1.28 (D5), U2.28 (D5), U3.28 (D5), U4.17 (D5), U5.23 (D5), U6.17 (D5)
- new net d6: U1.27 (D6), U2.27 (D6), U3.27 (D6), U4.18 (D6), U5.24 (D6), U6.18 (D6)
- new net d7: U1.26 (D7), U2.26 (D7), U3.26 (D7), U4.19 (D7), U5.25 (D7), U6.19 (D7)
- no-connect marks 0 -> 11

Commit message: schmatic updates
Parts:
- added C15: 0.1uF, Capacitor_THT:C_Disc_D3.4mm_W2.1mm_P2.50mm, symbol Device:C
- added C16: 2200uF, Capacitor_THT:C_Radial_D8.0mm_H7.0mm_P3.50mm, symbol Device:CP
- added D1, D2: LED, LED_THT:LED_D5.0mm_Clear, symbol Device:LED
- added J1: Jack-DC, Connector_BarrelJack:BarrelJack_Horizontal, symbol Connector:Jack-DC
- added R3, R4: 220, Resistor_THT:R_Axial_DIN0207_L6.3mm_D2.5mm_P7.62mm_Horizontal, symbol Device:R
- added U10: 74LS08, Package_DIP:DIP-14_W7.62mm_Socket, symbol 74xx:74LS08
- C1, C10, C11, C12, C13, C2, C3, C4, C5, C6, C7, C8, C9: footprint (none) -> Capacitor_THT:C_Disc_D3.4mm_W2.1mm_P2.50mm
- R1, R2: footprint (none) -> Resistor_THT:R_Axial_DIN0207_L6.3mm_D2.5mm_P7.62mm_Horizontal
- RV1: footprint (none) -> Potentiometer_THT:Potentiometer_Bourns_3296W_Vertical
- SW1: footprint (none) -> Button_Switch_THT:SW_PUSH_6mm_H4.3mm
- U1, U2: symbol 6502:65C22S -> 6502-rescue:65C22S-6502
- U3: symbol 6502:65C02S -> 6502-rescue:65C02S-6502
- U4: footprint Package_DIP:DIP-28_W15.24mm_Socket -> Socket:DIP_Socket-28_W11.9_W12.7_W15.24_W17.78_W18.5_3M_228-1277-00-0602J; symbol 6502:28C256 -> 6502-rescue:28C256-6502
- U5: symbol 6502:65C51N -> 6502-rescue:65C51N-6502
- U6: symbol 6502:62256 -> 6502-rescue:62256-6502
- U7, U9: footprint (none) -> Package_DIP:DIP-24_W7.62mm_Socket
- U8: footprint Display:NHD-0420H1Z -> 6502:LCD-20x4
- X1: value ACO-xxxMHz -> ACO-4MHz
- Y1: value Crystal -> 1.8432MHz; footprint (none) -> Crystal:Resonator-2Pin_W7.0mm_H2.5mm
Connections:
- net +5V: now also RV1.3, U8.2 (VDD), C15.2, C16.1, J1.1, R3.2, U10.14 (VCC)
- net 1pb0: now also U8.11 (DB4)
- net 1pb1: now also U8.12 (DB5)
- net 1pb2: now also U8.13 (DB6)
- net 1pb3: now also U8.14 (DB7)
- net 1pb4: now also U8.4 (RS)
- net 1pb5: now also U8.5 (R/W)
- net 1pb6: now also U8.6 (E)
- net 1pb7: now also R4.2
- net DEVICE_CS: now also U7.21 (O2/A1); no longer U7.18 (NC/O0)
- net GND: now also U5.9 (~CTS), U8.10 (DB3), U8.7 (DB0), U8.8 (DB1), U8.9 (DB2), C15.1, C16.2, D1.1 (K), D2.1 (K), J1.2, U10.7 (GND)
- net OE: now also U7.15 (A0/O3); no longer U7.14 (LR/O4)
- net RAM_CS: now also U7.18 (NC/O0); no longer U7.16 (A1/O2)
- net WE: now also U7.16 (A1/O2); no longer U7.15 (A0/O3)
- net a0: no longer U9.23 (A0)
- net a1: no longer U9.22 (A1)
- net a10: now also U7.9 (I7); no longer U7.8 (I6)
- net a11: now also U7.8 (I6); no longer U7.7 (I5)
- net a12: now also U7.7 (I5); no longer U7.6 (I4)
- net a13: now also U7.6 (I4); no longer U7.5 (I3)
- net a14: now also U7.5 (I3); no longer U7.4 (I2)
- net a2: no longer U9.21 (A2)
- net a3: no longer U9.20 (A3)
- net a4: now also U9.23 (A0)
- net a5: now also U9.22 (A1)
- net a6: now also U9.21 (A2)
- net a7: now also U9.20 (A3)
- net a8: now also U7.11 (I9); no longer U7.10 (I8)
- net a9: now also U7.10 (I8); no longer U7.9 (I7)
- net VP: now reaches U3.1 (~VP)
- net PHI1O: now reaches U3.3 (PHI1O)
- net IRQ: now reaches U3.4 (~IRQ)
- net IRQ: now also U10.6
- net ML: now reaches U3.5 (~ML)
- net SYNC: now reaches U3.7 (SYNC)
- net 1CB1: now reaches U2.18 (CB1)
- net 1CB2: now reaches U2.19 (CB2)
- net 1VIA_IRQ: now reaches U2.21 (~IRQ)
- net 1VIA_IRQ: now also U10.1
- net 1CA2: now reaches U2.39 (CA2)
- net 1CA1: now reaches U2.40 (CA1)
- net 2CB1: now reaches U1.18 (CB1)
- net 2CB2: now reaches U1.19 (CB2)
- net 2VIA_IRQ: now reaches U1.21 (~IRQ)
- net 2VIA_IRQ: now also U10.2
- net 2CA2: now reaches U1.39 (CA2)
- net 2CA1: now reaches U1.40 (CA1)
- net TxD: now reaches U5.10 (TxD)
- net RxD: now reaches U5.12 (RxD)
- net ACIA_IRQ: now reaches U5.26 (~IRQ)
- net ACIA_IRQ: now also U10.4
- net RTS: now reaches U5.8 (~RTS)
- net dev9: now reaches U9.10 (S9)
- net dev10: now reaches U9.11 (S10)
- net dev11: now reaches U9.13 (S11)
- net dev12: now reaches U9.14 (S12)
- net dev13: now reaches U9.15 (S13)
- net dev14: now reaches U9.16 (S14)
- net dev15: now reaches U9.17 (S15)
- net dev3: now reaches U9.4 (S3)
- net dev4: now reaches U9.5 (S4)
- net dev5: now reaches U9.6 (S5)
- net dev6: now reaches U9.7 (S6)
- net dev7: now reaches U9.8 (S7)
- net dev8: now reaches U9.9 (S8)
- net decode3: now reaches U7.19 (O4/NC)
- net decode2: now reaches U7.20 (O3/A2)
- net decode1: now reaches U7.22 (O1/A0)
- net decode0: now reaches U7.23 (O0/LR)
- new net: U10.3, U10.5
- new net: D1.2 (A), R3.1
- new net: D2.2 (A), R4.1
- new net decode4: U7.14 (LR/O4)
- no-connect marks 11 -> 4
Other:
- moved on the sheet: C13, R2, Y1

Commit message: changes
Parts:
- removed D2: LED, LED_THT:LED_D5.0mm_Clear, symbol Device:LED
- removed R4: 220, Resistor_THT:R_Axial_DIN0207_L6.3mm_D2.5mm_P7.62mm_Horizontal, symbol Device:R
- added C17: 0.1uF, Capacitor_THT:C_Disc_D3.4mm_W2.1mm_P2.50mm, symbol Device:C
- added unit 3 of U1
- added U4: 62256, Package_DIP:DIP-28_W15.24mm_Socket, symbol 6502-rescue:62256-6502
- renumbered C15 to C13, C13 to C14, C16 to C15, U10 to U1, U8 to U10, U5 to U11, U7 to U2, U9 to U3, U4 to U5, U3 to U6, U6 to U7, U1 to U8, U2 to U9
Connections:
- net decode4 is gone; now on net decode3: U2.14 (LR/O4)
- net +5V: now also C17.2, U4.28 (VCC)
- net 1pb7: now also U2.4 (I2)
- net ACIA_IRQ: now also U1.10
- net GND: now also C17.1, U4.14 (GND)
- net IRQ: now also U1.8; no longer U1.6
- net OE: now also U4.22 (~OE)
- net WE: now also U4.27 (~WE)
- net a0: now also U4.10 (A0)
- net a1: now also U4.9 (A1)
- net a10: now also U4.21 (A10)
- net a11: now also U4.23 (A11)
- net a12: now also U4.2 (A12)
- net a13: now also U4.26 (A13)
- net a14: now also U4.1 (A14)
- net a2: now also U4.8 (A2)
- net a3: now also U4.7 (A3)
- net a4: now also U4.6 (A4)
- net a5: now also U4.5 (A5)
- net a6: now also U4.4 (A6)
- net a7: now also U4.3 (A7)
- net a8: now also U4.25 (A8)
- net a9: now also U4.24 (A9)
- net d0: now also U4.11 (D0)
- net d1: now also U4.12 (D1)
- net d2: now also U4.13 (D2)
- net d3: now also U4.15 (D3)
- net d4: now also U4.16 (D4)
- net d5: now also U4.17 (D5)
- net d6: now also U4.18 (D6)
- net d7: now also U4.19 (D7)
- net decode3: no longer U2.19 (O4/NC)
- net RAM_CS renamed RAM_CS1
- new net: U1.6, U1.9
- new net RAM_CS2: U2.19 (O4/NC), U4.20 (~CE)
- no-connect marks 4 -> 3
Other:
- moved on the sheet: C13, RV1, U10, U1A, U1B, U7
