File: 6502/6502/interface.sch (KiCad schematic (older format))
At the start: 18 parts, among them J10 Conn_01x05, J11 DIN-6, J2 Conn_01x08, J3 Conn_01x08, J4 Conn_01x08, J5 Conn_01x16, J6 Conn_01x08, J7 Conn_01x08, J8 Conn_01x16, J9 Conn_01x06, U11 74HC14, U12 74HC595, U13 74HC595

Commit message: changes
Parts:
- removed J10: Conn_01x05, Connector_PinHeader_1.27mm:PinHeader_1x05_P1.27mm_Vertical, symbol Connector_Generic:Conn_01x05
- added J8: Conn_01x04, symbol Connector_Generic:Conn_01x04
- added unit 3 of U12
- renumbered C14 to C16, D3 to D2, J9 to J10, J3 to J2, J4 to J3, J2 to J4, J8 to J5, J5 to J6, J6 to J7, J7 to J9, R7 to R4, R6 to R5, R5 to R6, U11 to U12, U12 to U13, U13 to U14
Connections:
- net PS2_CLK: now also U12.5
- net decode0: now also J8.1 (Pin_1)
- net decode1: now also J8.2 (Pin_2)
- net decode2: now also J8.3 (Pin_3)
- net decode3: now also J8.4 (Pin_4)
- net at D2.2 (A), R4.1, U12.4: no longer U13.11 (SRCLK), U14.11 (SRCLK)
- new net: U12.6, U13.11 (SRCLK), U14.11 (SRCLK)
