File: 6502/interface.sch (KiCad schematic (older format))
At the start: 15 parts, among them J1 DB9_Female, J10 AudioJack2, J11 Mini-DIN-6, J12 Jack-DC, J13 Conn_01x08, J15 Conn_01x02, J17 Conn_01x02, J2 Conn_02x22_Odd_Even, J3 Conn_01x08, J4 Conn_02x22_Odd_Even, J5 Conn_02x22_Odd_Even, J6 Conn_02x22_Odd_Even, J7 Conn_01x06, J8 Conn_01x05, J9 Conn_01x08

Commit message: changes
Parts:
- removed J1: DB9_Female, symbol Connector:DB9_Female
- removed J10: AudioJack2, symbol Connector:AudioJack2
- removed J13: Conn_01x08, Connector_PinHeader_1.27mm:PinHeader_1x08_P1.27mm_Vertical, symbol Connector_Generic:Conn_01x08
- removed J2, J4, J5, J6: Conn_02x22_Odd_Even, symbol Connector_Generic:Conn_02x22_Odd_Even
- removed J7: Conn_01x06, symbol Connector_Generic:Conn_01x06
- added C17, C18: 1uF, Capacitor_THT:CP_Radial_D5.0mm_P2.50mm, symbol Device:CP
- added J10, J14, J2, J6: Conn_02x21_Odd_Even, Connector_PinHeader_1.27mm:PinHeader_2x21_P1.27mm_Vertical, symbol Connector_Generic:Conn_02x21_Odd_Even
- added J13: Conn_01x02, Connector_PinHeader_1.27mm:PinHeader_1x02_P1.27mm_Vertical, symbol Connector_Generic:Conn_01x02
- added J4: Conn_01x08, Connector_PinHeader_1.27mm:PinHeader_1x08_P1.27mm_Vertical, symbol Connector_Generic:Conn_01x08
- added J5: Conn_01x03, Connector_PinHeader_1.27mm:PinHeader_1x03_P1.27mm_Vertical, symbol Connector_Generic:Conn_01x03
- added Q1: FQP47P06, Package_TO_SOT_THT:TO-251-3-1EP_Horizontal_TabDown, symbol Device:Q_PMOS_GDS
- added U13: LM7805_TO220, Package_TO_SOT_THT:TO-251-3-1EP_Horizontal_TabDown, symbol Regulator_Linear:LM7805_TO220
- J11: footprint (none) -> 6502Computer:mini_din-6
- J15, J17: footprint (none) -> Connector_PinHeader_1.27mm:PinHeader_1x02_P1.27mm_Vertical
- J8: footprint (none) -> Connector_PinHeader_1.27mm:PinHeader_1x05_P1.27mm_Vertical
Connections:
- net +5V: now also C18.1, J10.39 (Pin_39), J10.40 (Pin_40), J14.39 (Pin_39), J14.40 (Pin_40), J2.39 (Pin_39), J2.40 (Pin_40), J6.39 (Pin_39), J6.40 (Pin_40), U13.3 (VO); no longer J12.1
- net 1pa4: now also J11.5; no longer J11.1
- net 1pa5: now also J11.1; no longer J11.5
- net BE: now also J10.28 (Pin_28), J14.28 (Pin_28), J2.28 (Pin_28), J6.28 (Pin_28)
- net GND: now also C17.2, C18.2, J10.41 (Pin_41), J10.42 (Pin_42), J14.41 (Pin_41), J14.42 (Pin_42), J2.41 (Pin_41), J2.42 (Pin_42), J6.41 (Pin_41), J6.42 (Pin_42), Q1.1 (G), U13.2 (GND)
- net IRQ: now also J10.26 (Pin_26), J14.26 (Pin_26), J2.26 (Pin_26), J6.26 (Pin_26)
- net ML: now also J10.34 (Pin_34), J14.34 (Pin_34), J2.34 (Pin_34), J6.34 (Pin_34)
- net NMI: now also J10.36 (Pin_36), J14.36 (Pin_36), J2.36 (Pin_36), J6.36 (Pin_36)
- net PHI1O: now also J10.38 (Pin_38), J14.38 (Pin_38), J2.38 (Pin_38), J6.38 (Pin_38)
- net PHI2: now also J10.20 (Pin_20), J14.20 (Pin_20), J2.20 (Pin_20), J6.20 (Pin_20)
- net RDY: now also J10.30 (Pin_30), J14.30 (Pin_30), J2.30 (Pin_30), J6.30 (Pin_30)
- net RESET: now also J10.22 (Pin_22), J14.22 (Pin_22), J2.22 (Pin_22), J6.22 (Pin_22)
- net RW: now also J10.18 (Pin_18), J14.18 (Pin_18), J2.18 (Pin_18), J6.18 (Pin_18)
- net SYNC: now also J10.24 (Pin_24), J14.24 (Pin_24), J2.24 (Pin_24), J6.24 (Pin_24)
- net VP: now also J10.32 (Pin_32), J14.32 (Pin_32), J2.32 (Pin_32), J6.32 (Pin_32)
- net a0: now also J10.1 (Pin_1), J14.1 (Pin_1), J2.1 (Pin_1), J6.1 (Pin_1)
- net a1: now also J10.3 (Pin_3), J14.3 (Pin_3), J2.3 (Pin_3), J6.3 (Pin_3)
- net a10: now also J10.21 (Pin_21), J14.21 (Pin_21), J2.21 (Pin_21), J6.21 (Pin_21)
- net a11: now also J10.23 (Pin_23), J14.23 (Pin_23), J2.23 (Pin_23), J6.23 (Pin_23)
- net a12: now also J10.25 (Pin_25), J14.25 (Pin_25), J2.25 (Pin_25), J6.25 (Pin_25)
- net a13: now also J10.27 (Pin_27), J14.27 (Pin_27), J2.27 (Pin_27), J6.27 (Pin_27)
- net a14: now also J10.29 (Pin_29), J14.29 (Pin_29), J2.29 (Pin_29), J6.29 (Pin_29)
- net a15: now also J10.31 (Pin_31), J14.31 (Pin_31), J2.31 (Pin_31), J6.31 (Pin_31)
- net a2: now also J10.5 (Pin_5), J14.5 (Pin_5), J2.5 (Pin_5), J6.5 (Pin_5)
- net a3: now also J10.7 (Pin_7), J14.7 (Pin_7), J2.7 (Pin_7), J6.7 (Pin_7)
- net a4: now also J10.9 (Pin_9), J14.9 (Pin_9), J2.9 (Pin_9), J6.9 (Pin_9)
- net a5: now also J10.11 (Pin_11), J14.11 (Pin_11), J2.11 (Pin_11), J6.11 (Pin_11)
- net a6: now also J10.13 (Pin_13), J14.13 (Pin_13), J2.13 (Pin_13), J6.13 (Pin_13)
- net a7: now also J10.15 (Pin_15), J14.15 (Pin_15), J2.15 (Pin_15), J6.15 (Pin_15)
- net a8: now also J10.17 (Pin_17), J14.17 (Pin_17), J2.17 (Pin_17), J6.17 (Pin_17)
- net a9: now also J10.19 (Pin_19), J14.19 (Pin_19), J2.19 (Pin_19), J6.19 (Pin_19)
- net d0: now also J10.2 (Pin_2), J14.2 (Pin_2), J2.2 (Pin_2), J6.2 (Pin_2)
- net d1: now also J10.4 (Pin_4), J14.4 (Pin_4), J2.4 (Pin_4), J6.4 (Pin_4)
- net d2: now also J10.6 (Pin_6), J14.6 (Pin_6), J2.6 (Pin_6), J6.6 (Pin_6)
- net d3: now also J10.8 (Pin_8), J14.8 (Pin_8), J2.8 (Pin_8), J6.8 (Pin_8)
- net d4: now also J10.10 (Pin_10), J14.10 (Pin_10), J2.10 (Pin_10), J6.10 (Pin_10)
- net d5: now also J10.12 (Pin_12), J14.12 (Pin_12), J2.12 (Pin_12), J6.12 (Pin_12)
- net d6: now also J10.14 (Pin_14), J14.14 (Pin_14), J2.14 (Pin_14), J6.14 (Pin_14)
- net d7: now also J10.16 (Pin_16), J14.16 (Pin_16), J2.16 (Pin_16), J6.16 (Pin_16)
- net dev10: now also J10.33 (Pin_33)
- net dev11: now also J10.35 (Pin_35)
- net dev12: now also J10.37 (Pin_37)
- net dev13: now also J14.33 (Pin_33)
- net dev14: now also J14.35 (Pin_35)
- net dev15: now also J14.37 (Pin_37)
- net dev4: now also J2.33 (Pin_33)
- net dev5: now also J2.35 (Pin_35)
- net dev6: now also J2.37 (Pin_37)
- net dev7: now also J6.33 (Pin_33)
- net dev8: now also J6.35 (Pin_35)
- net dev9: now also J6.37 (Pin_37)
- new net: J12.1, Q1.2 (D)
- new net: C17.1, Q1.3 (S), U13.1 (VI)
- new net 1pa6: J5.1 (Pin_1)
- new net 1pa7: J5.2 (Pin_2)
- new net 1pb[7..7]: J5.3 (Pin_3)
- new net 2pa0: J4.1 (Pin_1)
- new net 2pa1: J4.2 (Pin_2)
- new net 2pa2: J4.3 (Pin_3)
- new net 2pa3: J4.4 (Pin_4)
- new net 2pa4: J4.5 (Pin_5)
- new net 2pa5: J4.6 (Pin_6)
- new net 2pa6: J4.7 (Pin_7)
- new net 2pa7: J4.8 (Pin_8)
- new net dev2: J13.1 (Pin_1)
- new net dev3: J13.2 (Pin_2)
Other:
- moved on the sheet: J12, J17, J9

Commit message: updates!
Parts:
- removed J10, J14, J2, J6: Conn_02x21_Odd_Even, Connector_PinHeader_1.27mm:PinHeader_2x21_P1.27mm_Vertical, symbol Connector_Generic:Conn_02x21_Odd_Even
- added J1, J2, J6, J7: Conn_02x20_Odd_Even, Connector_PinHeader_2.54mm:PinHeader_2x20_P2.54mm_Vertical, symbol Connector_Generic:Conn_02x20_Odd_Even
- C17, C18: footprint Capacitor_THT:CP_Radial_D5.0mm_P2.50mm -> Capacitor_THT:C_Disc_D5.1mm_W3.2mm_P5.00mm
- J13, J15, J17: footprint Connector_PinHeader_1.27mm:PinHeader_1x02_P1.27mm_Vertical -> Connector_PinHeader_2.54mm:PinHeader_1x02_P2.54mm_Vertical
- J3, J4: footprint Connector_PinHeader_1.27mm:PinHeader_1x08_P1.27mm_Vertical -> Connector_PinHeader_2.54mm:PinHeader_1x08_P2.54mm_Vertical
- J5: footprint Connector_PinHeader_1.27mm:PinHeader_1x03_P1.27mm_Vertical -> Connector_PinHeader_2.54mm:PinHeader_1x03_P2.54mm_Vertical
- J8: footprint Connector_PinHeader_1.27mm:PinHeader_1x05_P1.27mm_Vertical -> Connector_PinHeader_2.54mm:PinHeader_1x05_P2.54mm_Vertical
- J9: footprint Connector_PinHeader_1.27mm:PinHeader_1x08_P1.27mm_Vertical -> Connector_PinHeader_2.54mm:PinHeader_1x05_P2.54mm_Vertical
Connections:
- net +5V: now also J1.39 (Pin_39), J2.39 (Pin_39), J6.39 (Pin_39), J7.39 (Pin_39)
- net BE: now also J1.28 (Pin_28), J2.28 (Pin_28), J6.28 (Pin_28), J7.28 (Pin_28)
- net GND: now also J1.40 (Pin_40), J2.40 (Pin_40), J6.40 (Pin_40), J7.40 (Pin_40)
- net IRQ: now also J1.26 (Pin_26), J2.26 (Pin_26), J6.26 (Pin_26), J7.26 (Pin_26)
- net ML: now also J1.34 (Pin_34), J2.34 (Pin_34), J6.34 (Pin_34), J7.34 (Pin_34)
- net NMI: now also J1.36 (Pin_36), J2.36 (Pin_36), J6.36 (Pin_36), J7.36 (Pin_36)
- net PHI1O: now also J1.38 (Pin_38), J2.38 (Pin_38), J6.38 (Pin_38), J7.38 (Pin_38)
- net PHI2: now also J1.20 (Pin_20), J2.20 (Pin_20), J6.20 (Pin_20), J7.20 (Pin_20)
- net RDY: now also J1.30 (Pin_30), J2.30 (Pin_30), J6.30 (Pin_30), J7.30 (Pin_30)
- net RESET: now also J1.22 (Pin_22), J2.22 (Pin_22), J6.22 (Pin_22), J7.22 (Pin_22)
- net RW: now also J1.18 (Pin_18), J2.18 (Pin_18), J6.18 (Pin_18), J7.18 (Pin_18)
- net SYNC: now also J1.24 (Pin_24), J2.24 (Pin_24), J6.24 (Pin_24), J7.24 (Pin_24)
- net VP: now also J1.32 (Pin_32), J2.32 (Pin_32), J6.32 (Pin_32), J7.32 (Pin_32)
- net a0: now also J1.1 (Pin_1), J2.1 (Pin_1), J6.1 (Pin_1), J7.1 (Pin_1)
- net a1: now also J1.3 (Pin_3), J2.3 (Pin_3), J6.3 (Pin_3), J7.3 (Pin_3)
- net a10: now also J1.21 (Pin_21), J2.21 (Pin_21), J6.21 (Pin_21), J7.21 (Pin_21)
- net a11: now also J1.23 (Pin_23), J2.23 (Pin_23), J6.23 (Pin_23), J7.23 (Pin_23)
- net a12: now also J1.25 (Pin_25), J2.25 (Pin_25), J6.25 (Pin_25), J7.25 (Pin_25)
- net a13: now also J1.27 (Pin_27), J2.27 (Pin_27), J6.27 (Pin_27), J7.27 (Pin_27)
- net a14: now also J1.29 (Pin_29), J2.29 (Pin_29), J6.29 (Pin_29), J7.29 (Pin_29)
- net a15: now also J1.31 (Pin_31), J2.31 (Pin_31), J6.31 (Pin_31), J7.31 (Pin_31)
- net a2: now also J1.5 (Pin_5), J2.5 (Pin_5), J6.5 (Pin_5), J7.5 (Pin_5)
- net a3: now also J1.7 (Pin_7), J2.7 (Pin_7), J6.7 (Pin_7), J7.7 (Pin_7)
- net a4: now also J1.9 (Pin_9), J2.9 (Pin_9), J6.9 (Pin_9), J7.9 (Pin_9)
- net a5: now also J1.11 (Pin_11), J2.11 (Pin_11), J6.11 (Pin_11), J7.11 (Pin_11)
- net a6: now also J1.13 (Pin_13), J2.13 (Pin_13), J6.13 (Pin_13), J7.13 (Pin_13)
- net a7: now also J1.15 (Pin_15), J2.15 (Pin_15), J6.15 (Pin_15), J7.15 (Pin_15)
- net a8: now also J1.17 (Pin_17), J2.17 (Pin_17), J6.17 (Pin_17), J7.17 (Pin_17)
- net a9: now also J1.19 (Pin_19), J2.19 (Pin_19), J6.19 (Pin_19), J7.19 (Pin_19)
- net d0: now also J1.2 (Pin_2), J2.2 (Pin_2), J6.2 (Pin_2), J7.2 (Pin_2)
- net d1: now also J1.4 (Pin_4), J2.4 (Pin_4), J6.4 (Pin_4), J7.4 (Pin_4)
- net d2: now also J1.6 (Pin_6), J2.6 (Pin_6), J6.6 (Pin_6), J7.6 (Pin_6)
- net d3: now also J1.8 (Pin_8), J2.8 (Pin_8), J6.8 (Pin_8), J7.8 (Pin_8)
- net d4: now also J1.10 (Pin_10), J2.10 (Pin_10), J6.10 (Pin_10), J7.10 (Pin_10)
- net d5: now also J1.12 (Pin_12), J2.12 (Pin_12), J6.12 (Pin_12), J7.12 (Pin_12)
- net d6: now also J1.14 (Pin_14), J2.14 (Pin_14), J6.14 (Pin_14), J7.14 (Pin_14)
- net d7: now also J1.16 (Pin_16), J2.16 (Pin_16), J6.16 (Pin_16), J7.16 (Pin_16)
- net dev10: now also J6.33 (Pin_33)
- net dev11: now also J6.35 (Pin_35)
- net dev12: now also J6.37 (Pin_37)
- net dev13: now also J7.33 (Pin_33)
- net dev14: now also J7.35 (Pin_35)
- net dev15: now also J7.37 (Pin_37)
- net dev4: now also J1.33 (Pin_33)
- net dev5: now also J1.35 (Pin_35)
- net dev6: now also J1.37 (Pin_37)
- net dev7: now also J2.33 (Pin_33)
- net dev8: now also J2.35 (Pin_35)
- net dev9: now also J2.37 (Pin_37)
Changed lines of the file:
@@
 F 0 "J8" H 3230 992 50  0000 L CNN
 F 1 "Conn_01x05" H 3230 901 50  0000 L CNN
-F 2 "Connector_PinHeader_1.27mm:PinHeader_1x05_P1.27mm_Vertical" H 3150 950 50  0001 C CNN
+F 2 "Connector_PinHeader_2.54mm:PinHeader_1x05_P2.54mm_Vertical" H 3150 950 50  0001 C CNN
 F 3 "~" H 3150 950 50  0001 C CNN
 	1    3150 950
@@
 F 0 "J3" H 1580 1042 50  0000 L CNN
 F 1 "Conn_01x08" H 1580 951 50  0000 L CNN
-F 2 "Connector_PinHeader_1.27mm:PinHeader_1x08_P1.27mm_Vertical" H 1500 1050 50  0001 C CNN
+F 2 "Connector_PinHeader_2.54mm:PinHeader_1x08_P2.54mm_Vertical" H 1500 1050 50  0001 C CNN
 F 3 "~" H 1500 1050 50  0001 C CNN
 	1    1500 1050
@@
 F 0 "J15" H 4480 842 50  0000 L CNN
 F 1 "Conn_01x02" H 4480 751 50  0000 L CNN
-F 2 "Connector_PinHeader_1.27mm:PinHeader_1x02_P1.27mm_Vertical" H 4400 850 50  0001 C CNN
+F 2 "Connector_PinHeader_2.54mm:PinHeader_1x02_P2.54mm_Vertical" H 4400 850 50  0001 C CNN
 F 3 "~" H 4400 850 50  0001 C CNN
 	1    4400 850
@@
 F 0 "J4" H 1580 1942 50  0000 L CNN
 F 1 "Conn_01x08" H 1580 1851 50  0000 L CNN
-F 2 "Connector_PinHeader_1.27mm:PinHeader_1x08_P1.27mm_Vertical" H 1500 1950 50  0001 C CNN
+F 2 "Connector_PinHeader_2.54mm:PinHeader_1x08_P2.54mm_Vertical" H 1500 1950 50  0001 C CNN
 F 3 "~" H 1500 1950 50  0001 C CNN
 	1    1500 1950
@@
 F 0 "J5" H 1580 2692 50  0000 L CNN
 F 1 "Conn_01x03" H 1580 2601 50  0000 L CNN
-F 2 "Connector_PinHeader_1.27mm:PinHeader_1x03_P1.27mm_Vertical" H 1500 2650 50  0001 C CNN
+F 2 "Connector_PinHeader_2.54mm:PinHeader_1x03_P2.54mm_Vertical" H 1500 2650 50  0001 C CNN
 F 3 "~" H 1500 2650 50  0001 C CNN
 	1    1500 2650
@@
 F 0 "C18" H 9968 1346 50  0000 L CNN
 F 1 "1uF" H 9968 1255 50  0000 L CNN
-F 2 "Capacitor_THT:CP_Radial_D5.0mm_P2.50mm" H 9888 1150 50  0001 C CNN
+F 2 "Capacitor_THT:C_Disc_D5.1mm_W3.2mm_P5.00mm" H 9888 1150 50  0001 C CNN
 F 3 "~" H 9850 1300 50  0001 C CNN
 	1    9850 1300
@@
 F 0 "C17" H 9118 1346 50  0000 L CNN
 F 1 "1uF" H 9118 1255 50  0000 L CNN
-F 2 "Capacitor_THT:CP_Radial_D5.0mm_P2.50mm" H 9038 1150 50  0001 C CNN
+F 2 "Capacitor_THT:C_Disc_D5.1mm_W3.2mm_P5.00mm" H 9038 1150 50  0001 C CNN
 F 3 "~" H 9000 1300 50  0001 C CNN
 	1    9000 1300
-	1    0    0    -1
-$EndComp
-$Comp
-L power:GND #PWR060
-U 1 1 63360F70
-P 1650 5450
-F 0 "#PWR060" H 1650 5200 50  0001 C CNN
-F 1 "GND" H 1655 5277 50  0000 C CNN
-F 2 "" H 1650 5450 50  0001 C CNN
-F 3 "" H 1650 5450 50  0001 C CNN
-	1    1650 5450
 	1    0    0    -1
 $EndComp
@@
 F 0 "J9" H 2830 1942 50  0000 L CNN
 F 1 "Conn_01x08" H 2830 1851 50  0000 L CNN
-F 2 "Connector_PinHeader_1.27mm:PinHeader_1x08_P1.27mm_Vertical" H 2750 1950 50  0001 C CNN
+F 2 "Connector_PinHeader_2.54mm:PinHeader_1x05_P2.54mm_Vertical" H 2750 1950 50  0001 C CNN
 F 3 "~" H 2750 1950 50  0001 C CNN
 	1    2750 1950
@@
 F 0 "J17" H 10430 1692 50  0000 L CNN
 F 1 "Conn_01x02" H 10430 1601 50  0000 L CNN
-F 2 "Connector_PinHeader_1.27mm:PinHeader_1x02_P1.27mm_Vertical" H 10350 1700 50  0001 C CNN
+F 2 "Connector_PinHeader_2.54mm:PinHeader_1x02_P2.54mm_Vertical" H 10350 1700 50  0001 C CNN
 F 3 "~" H 10350 1700 50  0001 C CNN
 	1    10350 1700
@@
 F 3 "" H 10150 1800 50  0001 C CNN
 	1    10150 1800
-	1    0    0    -1
-$EndComp
-$Comp
-L power:GND #PWR050
-U 1 1 631D1DCC
-P 3600 5450
-F 0 "#PWR050" H 3600 5200 50  0001 C CNN
-F 1 "GND" H 3605 5277 50  0000 C CNN
-F 2 "" H 3600 5450 50  0001 C CNN
-F 3 "" H 3600 5450 50  0001 C CNN
-	1    3600 5450
-	1    0    0    -1
-$EndComp
-$Comp
-L power:GND #PWR054
-U 1 1 631E4DCA
-P 5500 5450
-F 0 "#PWR054" H 5500 5200 50  0001 C CNN
-F 1 "GND" H 5505 5277 50  0000 C CNN
-F 2 "" H 5500 5450 50  0001 C CNN
-F 3 "" H 5500 5450 50  0001 C CNN
-	1    5500 5450
 	1    0    0    -1
 $EndComp
@@
 Entry Wire Line
 	8050 3450 8150 3550
-$Comp
-L power:GND #PWR064
-U 1 1 631F835E
-P 7350 5450
-F 0 "#PWR064" H 7350 5200 50  0001 C CNN
-F 1 "GND" H 7355 5277 50  0000 C CNN
-F 2 "" H 7350 5450 50  0001 C CNN
-F 3 "" H 7350 5450 50  0001 C CNN
-	1    7350 5450
-	1    0    0    -1
-$EndComp
 Text GLabel 4000 5950 0    50   Input ~ 0
 dev[2..3]
@@
 F 0 "J13" H 4630 6042 50  0000 L CNN
 F 1 "Conn_01x02" H 4630 5951 50  0000 L CNN
-F 2 "Connector_PinHeader_1.27mm:PinHeader_1x02_P1.27mm_Vertical" H 4550 6050 50  0001 C CNN
+F 2 "Connector_PinHeader_2.54mm:PinHeader_1x02_P2.54mm_Vertical" H 4550 6050 50  0001 C CNN
 F 3 "~" H 4550 6050 50  0001 C CNN
 	1    4550 6050
@@
 L power:GND #PWR066
 U 1 1 631F8358
-P 7850 5450
-F 0 "#PWR066" H 7850 5200 50  0001 C CNN
-F 1 "GND" H 7855 5277 50  0000 C CNN
-F 2 "" H 7850 5450 50  0001 C CNN
-F 3 "" H 7850 5450 50  0001 C CNN
-	1    7850 5450
-	1    0    0    -1
-$EndComp
-$Comp
-L power:+5V #PWR065
-U 1 1 631F834C
 P 7850 5350
-F 0 "#PWR065" H 7850 5200 50  0001 C CNN
-F 1 "+5V" H 7865 5523 50  0000 C CNN
+F 0 "#PWR066" H 7850 5100 50  0001 C CNN
+F 1 "GND" H 7855 5177 50  0000 C CNN
 F 2 "" H 7850 5350 50  0001 C CNN
 F 3 "" H 7850 5350 50  0001 C CNN
 	1    7850 5350
-	0    1    1    0
+	1    0    0    -1
 $EndComp
 $Comp
 L power:GND #PWR059
 U 1 1 631E4DC4
-P 6000 5450
-F 0 "#PWR059" H 6000 5200 50  0001 C CNN
-F 1 "GND" H 6005 5277 50  0000 C CNN
-F 2 "" H 6000 5450 50  0001 C CNN
-F 3 "" H 6000 5450 50  0001 C CNN
-	1    6000 5450
-	1    0    0    -1
-$EndComp
-$Comp
-L power:+5V #PWR055
-U 1 1 631E4DB8
 P 6000 5350
-F 0 "#PWR055" H 6000 5200 50  0001 C CNN
-F 1 "+5V" H 6015 5523 50  0000 C CNN
+F 0 "#PWR059" H 6000 5100 50  0001 C CNN
+F 1 "GND" H 6005 5177 50  0000 C CNN
 F 2 "" H 6000 5350 50  0001 C CNN
 F 3 "" H 6000 5350 50  0001 C CNN
 	1    6000 5350
-	0    1    1    0
+	1    0    0    -1
 $EndComp
 $Comp
 L power:GND #PWR052
 U 1 1 631D1DC6
-P 4100 5450
-F 0 "#PWR052" H 4100 5200 50  0001 C CNN
-F 1 "GND" H 4105 5277 50  0000 C CNN
-F 2 "" H 4100 5450 50  0001 C CNN
-F 3 "" H 4100 5450 50  0001 C CNN
-	1    4100 5450
-	1    0    0    -1
-$EndComp
-$Comp
-L power:+5V #PWR051
-U 1 1 631D1DBA
 P 4100 5350
-F 0 "#PWR051" H 4100 5200 50  0001 C CNN
-F 1 "+5V" H 4115 5523 50  0000 C CNN
+F 0 "#PWR052" H 4100 5100 50  0001 C CNN
+F 1 "GND" H 4105 5177 50  0000 C CNN
 F 2 "" H 4100 5350 50  0001 C CNN
 F 3 "" H 4100 5350 50  0001 C CNN
 	1    4100 5350
-	0    1    1    0
+	1    0    0    -1
 $EndComp
 $Comp
 L power:GND #PWR063
 U 1 1 63360F6A
-P 2150 5450
-F 0 "#PWR063" H 2150 5200 50  0001 C CNN
-F 1 "GND" H 2155 5277 50  0000 C CNN
-F 2 "" H 2150 5450 50  0001 C CNN
-F 3 "" H 2150 5450 50  0001 C CNN
-	1    2150 5450
-	1    0    0    -1
-$EndComp
-$Comp
-L power:+5V #PWR070
-U 1 1 63499170
 P 2150 5350
-F 0 "#PWR070" H 2150 5200 50  0001 C CNN
-F 1 "+5V" H 2165 5523 50  0000 C CNN
+F 0 "#PWR063" H 2150 5100 50  0001 C CNN
+F 1 "GND" H 2155 5177 50  0000 C CNN
 F 2 "" H 2150 5350 50  0001 C CNN
 F 3 "" H 2150 5350 50  0001 C CNN
 	1    2150 5350
-	0    1    1    0
-$EndComp
-$Comp
-L Connector_Generic:Conn_02x21_Odd_Even J14
-U 1 1 631F8364
-P 7550 4450
-F 0 "J14" H 7600 5667 50  0000 C CNN
-F 1 "Conn_02x21_Odd_Even" H 7600 5576 50  0000 C CNN
-F 2 "Connector_PinHeader_1.27mm:PinHeader_2x21_P1.27mm_Vertical" H 7550 4450 50  0001 C CNN
-F 3 "~" H 7550 4450 50  0001 C CNN
-	1    7550 4450
-	1    0    0    -1
-$EndComp
-$Comp
-L Connector_Generic:Conn_02x21_Odd_Even J10
-U 1 1 631E4DD0
-P 5700 4450
-F 0 "J10" H 5750 5667 50  0000 C CNN
-F 1 "Conn_02x21_Odd_Even" H 5750 5576 50  0000 C CNN
-F 2 "Connector_PinHeader_1.27mm:PinHeader_2x21_P1.27mm_Vertical" H 5700 4450 50  0001 C CNN
-F 3 "~" H 5700 4450 50  0001 C CNN
-	1    5700 4450
-	1    0    0    -1
-$EndComp
-$Comp
-L Connector_Generic:Conn_02x21_Odd_Even J6
-U 1 1 631D1DD2
-P 3800 4450
-F 0 "J6" H 3850 5667 50  0000 C CNN
-F 1 "Conn_02x21_Odd_Even" H 3850 5576 50  0000 C CNN
-F 2 "Connector_PinHeader_1.27mm:PinHeader_2x21_P1.27mm_Vertical" H 3800 4450 50  0001 C CNN
-F 3 "~" H 3800 4450 50  0001 C CNN
-	1    3800 4450
-	1    0    0    -1
-$EndComp
-$Comp
-L Connector_Generic:Conn_02x21_Odd_Even J2
-U 1 1 630D8C84
-P 1850 4450
-F 0 "J2" H 1900 5667 50  0000 C CNN
-F 1 "Conn_02x21_Odd_Even" H 1900 5576 50  0000 C CNN
-F 2 "Connector_PinHeader_1.27mm:PinHeader_2x21_P1.27mm_Vertical" H 1850 4450 50  0001 C CNN
-F 3 "~" H 1850 4450 50  0001 C CNN
-	1    1850 4450
-	1    0    0    -1
-$EndComp
+	1    0    0    -1
+$EndComp
+$Comp
+L Connector_Generic:Conn_02x20_Odd_Even J1
+U 1 1 63011402
+P 1850 4350
+F 0 "J1" H 1900 5467 50  0000 C CNN
+F 1 "Conn_02x20_Odd_Even" H 1900 5376 50  0000 C CNN
+F 2 "Connector_PinHeader_2.54mm:PinHeader_2x20_P2.54mm_Vertical" H 1850 4350 50  0001 C CNN
+F 3 "~" H 1850 4350 50  0001 C CNN
+	1    1850 4350
+	1    0    0    -1
+$EndComp
+$Comp
+L Connector_Generic:Conn_02x20_Odd_Even J2
+U 1 1 63041508
+P 3800 4350
+F 0 "J2" H 3850 5467 50  0000 C CNN
+F 1 "Conn_02x20_Odd_Even" H 3850 5376 50  0000 C CNN
+F 2 "Connector_PinHeader_2.54mm:PinHeader_2x20_P2.54mm_Vertical" H 3800 4350 50  0001 C CNN
+F 3 "~" H 3800 4350 50  0001 C CNN
+	1    3800 4350
+	1    0    0    -1
+$EndComp
+$Comp
+L Connector_Generic:Conn_02x20_Odd_Even J6
+U 1 1 63043AFA
+P 5700 4350
+F 0 "J6" H 5750 5467 50  0000 C CNN
+F 1 "Conn_02x20_Odd_Even" H 5750 5376 50  0000 C CNN
+F 2 "Connector_PinHeader_2.54mm:PinHeader_2x20_P2.54mm_Vertical" H 5700 4350 50  0001 C CNN
+F 3 "~" H 5700 4350 50  0001 C CNN
+	1    5700 4350
+	1    0    0    -1
+$EndComp
+$Comp
+L Connector_Generic:Conn_02x20_Odd_Even J7
+U 1 1 63044A49
+P 7550 4350
+F 0 "J7" H 7600 5467 50  0000 C CNN
+F 1 "Conn_02x20_Odd_Even" H 7600 5376 50  0000 C CNN
+F 2 "Connector_PinHeader_2.54mm:PinHeader_2x20_P2.54mm_Vertical" H 7550 4350 50  0001 C CNN
+F 3 "~" H 7550 4350 50  0001 C CNN
+	1    7550 4350
+	1    0    0    -1
+$EndComp
