File: 6502/6502.kicad_pcb (KiCad board)
At the start: 2 copper layers, 54 parts, among them J1 Jack-DC, J10 Conn_01x05, J11 DIN-6, J2 Conn_01x08, J3 Conn_01x08, J4 Conn_01x08, J5 Conn_01x16, J6 Conn_01x08, J7 Conn_01x08, J8 Conn_01x16, J9 Conn_01x06, SW1 SW_Push, U1 65C22S, U10 74LS08, U11 74HC14, U12 74HC595, U13 74HC595, U2 65C22S, U3 65C02S, U4 28C256, U5 65C51N, U6 62256, U7 PAL24, U8 NHD-0420H1Z, U9 74LS154, X1 ACO-4MHz, Y1 1.8432MHz

Commit message: changes
Parts:
- removed C10, C11, C12, C14: 0.1uF, Capacitor_THT:C_Disc_D3.4mm_W2.1mm_P2.50mm
- removed C13: 30pF, Capacitor_THT:C_Disc_D3.4mm_W2.1mm_P2.50mm
- removed D2: LED, LED_THT:LED_D5.0mm_Clear
- removed D3: 5.1V, Diode_THT:D_A-405_P7.62mm_Horizontal
- removed J1: Jack-DC, Connector_BarrelJack:BarrelJack_Horizontal
- removed J7: Conn_01x08, Connector_PinHeader_1.27mm:PinHeader_1x08_P1.27mm_Vertical
- removed U11: 74HC14, Package_DIP:DIP-14_W7.62mm_Socket
- removed U6: 62256, Package_DIP:DIP-28_W15.24mm_Socket
- removed U9: 74LS154, Package_DIP:DIP-24_W7.62mm_Socket
- removed Y1: 1.8432MHz, Crystal:Resonator-2Pin_W7.0mm_H2.5mm
- added C17: 1uF, Capacitor_THT:CP_Radial_D5.0mm_P2.50mm, F.Cu at (-44.1, 41.9)
- added C18: 1uF, Capacitor_THT:CP_Radial_D5.0mm_P2.50mm, F.Cu at (-50.7, 44.0)
- added J12: Jack-DC, Connector_BarrelJack:BarrelJack_Horizontal, F.Cu at (-55.4, 33.9)
- added J13: Conn_01x02, Connector_PinHeader_1.27mm:PinHeader_1x02_P1.27mm_Vertical, F.Cu at (-81.5, 43.8)
- added J14: Conn_02x21_Odd_Even, Connector_PinHeader_1.27mm:PinHeader_2x21_P1.27mm_Vertical, F.Cu at (-89.8, 15.1)
- added J15: Conn_01x02, Connector_PinHeader_1.27mm:PinHeader_1x02_P1.27mm_Vertical, F.Cu at (-85.7, 43.8)
- added J17: Conn_01x02, Connector_PinHeader_1.27mm:PinHeader_1x02_P1.27mm_Vertical, F.Cu at (-89.8, 43.8)
- added Q1: FQP47P06, Package_TO_SOT_THT:TO-251-3-1EP_Horizontal_TabDown, F.Cu at (-42.0, 24.7)
- added R8: 1K, Resistor_THT:R_Axial_DIN0207_L6.3mm_D2.5mm_P7.62mm_Horizontal, F.Cu at (-35.7, -29.5)
- added R9: 1K, Resistor_THT:R_Axial_DIN0207_L6.3mm_D2.5mm_P7.62mm_Horizontal, F.Cu at (-47.4, -14.0)
- added SW2: SW_Push, Button_Switch_THT:SW_PUSH_6mm_H4.3mm, F.Cu at (-47.0, -9.97)
- C15: value 0.1uF -> 2200uF; footprint Capacitor_THT:C_Disc_D3.4mm_W2.1mm_P2.50mm -> Capacitor_THT:C_Radial_D8.0mm_H7.0mm_P3.50mm
- C16: value 2200uF -> 0.1uF; footprint Capacitor_THT:C_Radial_D8.0mm_H7.0mm_P3.50mm -> Capacitor_THT:C_Disc_D3.4mm_W2.1mm_P2.50mm
- J10: value Conn_01x05 -> Conn_02x21_Odd_Even; footprint Connector_PinHeader_1.27mm:PinHeader_1x05_P1.27mm_Vertical -> Connector_PinHeader_1.27mm:PinHeader_2x21_P1.27mm_Vertical
- J11: value DIN-6 -> Mini-DIN-6; footprint 6502:mini_din-6 -> 6502Computer:mini_din-6
- J2, J6: value Conn_01x08 -> Conn_02x21_Odd_Even; footprint Connector_PinHeader_1.27mm:PinHeader_1x08_P1.27mm_Vertical -> Connector_PinHeader_1.27mm:PinHeader_2x21_P1.27mm_Vertical
- J5: value Conn_01x16 -> Conn_01x03; footprint Connector_PinHeader_1.27mm:PinHeader_1x16_P1.27mm_Vertical -> Connector_PinHeader_1.27mm:PinHeader_1x03_P1.27mm_Vertical
- J8: value Conn_01x16 -> Conn_01x05; footprint Connector_PinHeader_1.27mm:PinHeader_1x16_P1.27mm_Vertical -> Connector_PinHeader_1.27mm:PinHeader_1x05_P1.27mm_Vertical
- J9: value Conn_01x06 -> Conn_01x08; footprint Connector_PinHeader_1.27mm:PinHeader_1x06_P1.27mm_Vertical -> Connector_PinHeader_1.27mm:PinHeader_1x08_P1.27mm_Vertical
- R2: value 1M -> 1K
- R3: value 220 -> 220Ω
- R4: value 220 -> 1K
- R7: value 21K -> 10K
- U1: value 65C22S -> 74LS08; footprint Package_DIP:DIP-40_W15.24mm_Socket -> Package_DIP:DIP-14_W7.62mm_Socket
- U10: value 74LS08 -> NHD-0420H1Z; footprint Package_DIP:DIP-14_W7.62mm_Socket -> 6502Computer:LCD-20x4
- U12: value 74HC595 -> 65C02S; footprint Package_DIP:DIP-16_W7.62mm_Socket -> Package_DIP:DIP-40_W15.24mm_Socket
- U13: value 74HC595 -> LM7805_TO220; footprint Package_DIP:DIP-16_W7.62mm_Socket -> Package_TO_SOT_THT:TO-251-3-1EP_Horizontal_TabDown
- U2: value 65C22S -> PAL24; footprint Package_DIP:DIP-40_W15.24mm_Socket -> Package_DIP:DIP-24_W7.62mm_Socket
- U3: value 65C02S -> 74LS154; footprint Package_DIP:DIP-40_W15.24mm_Socket -> Package_DIP:DIP-24_W7.62mm_Socket
- U4: value 28C256 -> AS6C4008-55PCN; footprint Socket:DIP_Socket-28_W11.9_W12.7_W15.24_W17.78_W18.5_3M_228-1277-00-0602J -> Package_DIP:DIP-32_W15.24mm_Socket
- U5: value 65C51N -> 28C256; footprint Package_DIP:DIP-28_W15.24mm_Socket -> 6502Computer:ZIF_Socket-28
- U7: value PAL24 -> 6522; footprint Package_DIP:DIP-24_W7.62mm_Socket -> Package_DIP:DIP-40_W15.24mm_Socket
- U8: value NHD-0420H1Z -> 6522; footprint 6502:LCD-20x4 -> Package_DIP:DIP-40_W15.24mm_Socket
- moved R7 236.0 mm to (-70.9, 2.05)
- moved J10 235.9 mm to (-73.3, 15.1)
- moved R5 228.8 mm to (-70.9, 6.10)
- moved J6 228.7 mm to (-84.3, 15.1)
- moved C5 218.7 mm to (-60.2, 8.58)
- moved C6 217.3 mm to (-35.7, -17.9)
- moved J2 216.1 mm to (-78.8, 15.1)
- moved U10 216.0 mm to (-0.44, 97.2)
- moved C3 206.0 mm to (-35.7, -21.6)
- moved C4 205.9 mm to (-60.2, 4.93)
- moved C7 201.8 mm to (-30.0, -21.1)
- moved C1 198.9 mm to (-13.1, -33.7)
- moved R3 195.8 mm to (-35.7, -25.4)
- moved J11 195.0 mm to (-59.6, 19.0)
- moved D1 194.7 mm to (-37.6, 0.33)
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Connections:
- C15 pad 1: GND -> +5V
- C15 pad 2: +5V -> GND
- C16 pad 1: +5V -> NMI
- J10 pad 1: decode0 -> a0
- J10 pad 2: decode1 -> d0
- J10 pad 3: decode2 -> a1
- J10 pad 4: decode3 -> d1
- J10 pad 5: decode4 -> a2
- J11 pad 1: PS2_D -> 1pa5
- J11 pad 5: PS2_CLK -> 1pa4
- J2 pad 1: 2pa0 -> a0
- J2 pad 2: 2pa1 -> d0
- J2 pad 3: 2pa2 -> a1
- J2 pad 4: 2pa3 -> d1
- J2 pad 5: 2pa4 -> a2
- J2 pad 6: 2pa5 -> d2
- J2 pad 7: 2pa6 -> a3
- J2 pad 8: 2pa7 -> d3
- J3 pad 1: d7 -> 2pb0
- J3 pad 2: d6 -> 2pb1
- J3 pad 3: d5 -> 2pb2
- J3 pad 4: d4 -> 2pb3
- J3 pad 5: d3 -> 2pb4
- J3 pad 6: d2 -> 2pb5
- J3 pad 7: d1 -> 2pb6
- J3 pad 8: d0 -> 2pb7
- J4 pad 1: 2pb0 -> 2pa0
- J4 pad 2: 2pb1 -> 2pa1
- J4 pad 3: 2pb2 -> 2pa2
- J4 pad 4: 2pb3 -> 2pa3
- J4 pad 5: 2pb4 -> 2pa4
- J4 pad 6: 2pb5 -> 2pa5
- J4 pad 7: 2pb6 -> 2pa6
- J4 pad 8: 2pb7 -> 2pa7
- J5 pad 1: a0 -> 1pa6
- J5 pad 2: a1 -> 1pa7
- J5 pad 3: a2 -> 1pb7
- J6 pad 1: PHI2 -> a0
- J6 pad 2: VP -> d0
- J6 pad 3: PHI1O -> a1
- J6 pad 4: IRQ -> d1
- J6 pad 5: ML -> a2
- J6 pad 6: SYNC -> d2
- J6 pad 7: RW -> a3
- J6 pad 8: RESET -> d3
- J8 pad 1: dev15 -> decode0
- J8 pad 2: dev14 -> decode1
- J8 pad 3: dev13 -> decode2
- J8 pad 4: dev12 -> decode3
- J8 pad 5: dev11 -> decode4
- J9 pad 1: GND -> 1CB1
- J9 pad 2: TxD -> 1CB2
- J9 pad 3: RxD -> 1CA1
- J9 pad 4: +5V -> 1CA2
- J9 pad 5: RTS -> 2CB1
- J9 pad 6: GND -> 2CB2
- R2 pad 1: Net-(C13-Pad1) -> 1pa0
- R2 pad 2: Net-(R2-Pad2) -> GND
- R4 pad 1: Net-(D2-Pad2) -> 1pa1
- R4 pad 2: 1pb7 -> GND
- R5 pad 1: Net-(R5-Pad1) -> +5V
- R5 pad 2: +5V -> RDY
- R6 pad 1: Net-(R6-Pad1) -> BE
- R7 pad 1: Net-(D3-Pad2) -> +5V
- R7 pad 2: Net-(C14-Pad1) -> NMI
- U1 pad 1: GND -> 1VIA_IRQ
- U1 pad 10: 2pb0 -> (no net)
- U1 pad 11: 2pb1 -> (no net)
- U1 pad 12: 2pb2 -> (no net)
- U1 pad 13: 2pb3 -> (no net)
- U1 pad 14: 2pb4 -> +5V
- U1 pad 2: 2pa0 -> 2VIA_IRQ
- U1 pad 3: 2pa1 -> IRQ
- U1 pad 4: 2pa2 -> (no net)
- U1 pad 5: 2pa3 -> (no net)
- U1 pad 6: 2pa4 -> (no net)
- U1 pad 7: 2pa5 -> GND
- U1 pad 8: 2pa6 -> (no net)
- U1 pad 9: 2pa7 -> (no net)
- U10 pad 1: 1VIA_IRQ -> GND
- U10 pad 10: (no net) -> GND
- U10 pad 11: (no net) -> 1pb0
- U10 pad 12: (no net) -> 1pb1
- U10 pad 13: (no net) -> 1pb2
- U10 pad 14: +5V -> 1pb3
- U10 pad 2: 2VIA_IRQ -> +5V
- U10 pad 3: Net-(U10-Pad3) -> Net-(RV1-Pad2)
- U10 pad 4: ACIA_IRQ -> 1pb4
- U10 pad 5: Net-(U10-Pad3) -> 1pb5
- U10 pad 6: IRQ -> 1pb6
- U10 pad 8: (no net) -> GND
- U10 pad 9: (no net) -> GND
- U12 pad 1: Net-(U12-Pad1) -> VP
- U12 pad 10: Net-(R6-Pad1) -> a1
- U12 pad 11: Net-(U11-Pad6) -> a2
- U12 pad 12: 1CA1 -> a3
- U12 pad 13: GND -> a4
- U12 pad 14: PS2_D -> a5
- U12 pad 15: Net-(U12-Pad15) -> a6
- U12 pad 16: +5V -> a7
- U12 pad 2: 1pa7 -> RDY
- U12 pad 3: 1pa6 -> PHI1O
- U12 pad 4: 1pa5 -> IRQ
- U12 pad 5: 1pa4 -> ML
- U12 pad 6: 1pa3 -> NMI
- U12 pad 7: 1pa2 -> SYNC
- U12 pad 8: GND -> +5V
- U12 pad 9: Net-(U12-Pad9) -> a0
- U13 pad 1: 1pa0 -> Net-(C17-Pad1)
- U13 pad 2: Net-(U13-Pad2) -> GND
- U13 pad 3: Net-(U13-Pad3) -> +5V
- U13 pad 4: Net-(U13-Pad4) -> (no net)
- U2 pad 1: GND -> PHI2
- U2 pad 10: 1pb0 -> a9
- U2 pad 11: 1pb1 -> a8
- U2 pad 12: 1pb2 -> GND
- U2 pad 13: 1pb3 -> EXT_IN1
- U2 pad 14: 1pb4 -> decode4
- U2 pad 15: 1pb5 -> OE
- U2 pad 16: 1pb6 -> WE
- U2 pad 17: 1pb7 -> ROM_CS
- U2 pad 18: 1CB1 -> RAM_CS
- U2 pad 19: 1CB2 -> decode3
- U2 pad 2: 1pa0 -> RW
- U2 pad 20: +5V -> decode2
- U2 pad 21: 1VIA_IRQ -> DEVICE_CS
- U2 pad 22: RW -> decode1
- U2 pad 23: VIA1_CS -> decode0
- U2 pad 3: 1pa1 -> EXT_IN2
- U2 pad 4: 1pa2 -> EXT_IN2
- U2 pad 5: 1pa3 -> a14
- U2 pad 6: 1pa4 -> a13
- U2 pad 7: 1pa5 -> a12
- U2 pad 8: 1pa6 -> a11
- U2 pad 9: 1pa7 -> a10
- U3 pad 1: VP -> VIA1_CS
- U3 pad 10: a1 -> dev9
- U3 pad 11: a2 -> dev10
- U3 pad 12: a3 -> GND
- U3 pad 13: a4 -> dev11
- U3 pad 14: a5 -> dev12
- U3 pad 15: a6 -> dev13
- U3 pad 16: a7 -> dev14
- U3 pad 17: a8 -> dev15
- U3 pad 18: a9 -> EXT_IN2
- U3 pad 19: a10 -> DEVICE_CS
- U3 pad 2: +5V -> VIA2_CS
- U3 pad 20: a11 -> a7
- U3 pad 21: GND -> a6
- U3 pad 22: a12 -> a5
- U3 pad 23: a13 -> a4
- U3 pad 24: a14 -> +5V
- U3 pad 3: PHI1O -> dev2
- U3 pad 4: IRQ -> dev3
- U3 pad 5: ML -> dev4
- U3 pad 6: +5V -> dev5
- U3 pad 7: SYNC -> dev6
- U3 pad 8: +5V -> dev7
- U3 pad 9: a0 -> dev8
- U4 pad 1: a14 -> 1pa3
- U4 pad 10: a0 -> a2
- U4 pad 11: d0 -> a1
- U4 pad 12: d1 -> a0
- U4 pad 13: d2 -> d0
- U4 pad 14: GND -> d1
- U4 pad 15: d3 -> d2
- U4 pad 16: d4 -> GND
- U4 pad 17: d5 -> d3
- U4 pad 18: d6 -> d4
- U4 pad 19: d7 -> d5
- U4 pad 2: a12 -> 1pa1
- U4 pad 20: ROM_CS -> d6
- U4 pad 21: a10 -> d7
- U4 pad 22: OE -> RAM_CS
- U4 pad 23: a11 -> a10
- U4 pad 24: a9 -> OE
- U4 pad 25: a8 -> a11
- U4 pad 26: a13 -> a9
- U4 pad 27: WE -> a8
- U4 pad 28: +5V -> a13
- U4 pad 3: a7 -> a14
- U4 pad 4: a6 -> a12
- U4 pad 5: a5 -> a7
- U4 pad 6: a4 -> a6
- U4 pad 7: a3 -> a5
- U4 pad 8: a2 -> a4
- U4 pad 9: a1 -> a3
- U5 pad 1: GND -> a14
- U5 pad 10: TxD -> a0
- U5 pad 11: Net-(U5-Pad11) -> d0
- U5 pad 12: RxD -> d1
- U5 pad 13: a0 -> d2
- U5 pad 14: a1 -> GND
- U5 pad 15: +5V -> d3
- U5 pad 16: Net-(U5-Pad11) -> d4
- U5 pad 17: Net-(U5-Pad11) -> d5
- U5 pad 18: d0 -> d6
- U5 pad 19: d1 -> d7
- U5 pad 2: +5V -> a12
- U5 pad 20: d2 -> ROM_CS
- U5 pad 21: d3 -> a10
- U5 pad 22: d4 -> OE
- U5 pad 23: d5 -> a11
- U5 pad 24: d6 -> a9
- U5 pad 25: d7 -> a8
- U5 pad 26: ACIA_IRQ -> a13
- U5 pad 27: PHI2 -> WE
- U5 pad 28: RW -> +5V
- U5 pad 3: ACIA_CS -> a7
- U5 pad 4: RESET -> a6
- U5 pad 5: Net-(U5-Pad5) -> a5
- U5 pad 6: Net-(C13-Pad1) -> a4
- U5 pad 7: Net-(R2-Pad2) -> a3
- U5 pad 8: RTS -> a2
- U5 pad 9: GND -> a1
- U7 pad 1: PHI2 -> GND
- U7 pad 10: a9 -> 2pb0
- U7 pad 11: a8 -> 2pb1
- U7 pad 12: GND -> 2pb2
- U7 pad 13: Net-(U7-Pad13) -> 2pb3
- U7 pad 14: decode4 -> 2pb4
- U7 pad 15: OE -> 2pb5
- U7 pad 16: WE -> 2pb6
- U7 pad 17: ROM_CS -> 2pb7
- U7 pad 18: RAM_CS -> 2CB1
- U7 pad 19: decode3 -> 2CB2
- U7 pad 2: RW -> 2pa0
- U7 pad 20: decode2 -> +5V
- U7 pad 21: DEVICE_CS -> 2VIA_IRQ
- U7 pad 22: decode1 -> RW
- U7 pad 23: decode0 -> VIA2_CS
- U7 pad 3: a15 -> 2pa1
- U7 pad 4: Net-(U7-Pad4) -> 2pa2
- U7 pad 5: a14 -> 2pa3
- U7 pad 6: a13 -> 2pa4
- U7 pad 7: a12 -> 2pa5
- U7 pad 8: a11 -> 2pa6
- U7 pad 9: a10 -> 2pa7
- U8 pad 10: GND -> 1pb0
- U8 pad 11: 1pb0 -> 1pb1
- U8 pad 12: 1pb1 -> 1pb2
- U8 pad 13: 1pb2 -> 1pb3
- U8 pad 14: 1pb3 -> 1pb4
- U8 pad 15: +5V -> 1pb5
- U8 pad 16: GND -> 1pb6
- U8 pad 2: +5V -> 1pa0
- U8 pad 3: Net-(RV1-Pad2) -> 1pa1
- U8 pad 4: 1pb4 -> 1pa2
- U8 pad 5: 1pb5 -> 1pa3
- U8 pad 6: 1pb6 -> 1pa4
- U8 pad 7: GND -> 1pa5
- U8 pad 8: GND -> 1pa6
- U8 pad 9: GND -> 1pa7

Commit message: worked on pcb
Parts:
- removed J10, J14: Conn_02x21_Odd_Even, Connector_PinHeader_1.27mm:PinHeader_2x21_P1.27mm_Vertical
- added J1: Conn_02x20_Odd_Even, Connector_PinHeader_2.54mm:PinHeader_2x20_P2.54mm_Vertical, F.Cu at (153.9, 80.3)
- added J7: Conn_02x20_Odd_Even, Connector_PinHeader_2.54mm:PinHeader_2x20_P2.54mm_Vertical, F.Cu at (132.0, 80.0)
- C1, C16, C2, C3, C4, C5, C6, C7, C8, C9: footprint Capacitor_THT:C_Disc_D3.4mm_W2.1mm_P2.50mm -> Capacitor_THT:C_Disc_D5.1mm_W3.2mm_P5.00mm
- C17, C18: footprint Capacitor_THT:CP_Radial_D5.0mm_P2.50mm -> Capacitor_THT:C_Disc_D5.1mm_W3.2mm_P5.00mm
- J13, J15, J17: footprint Connector_PinHeader_1.27mm:PinHeader_1x02_P1.27mm_Vertical -> Connector_PinHeader_2.54mm:PinHeader_1x02_P2.54mm_Vertical
- J2, J6: value Conn_02x21_Odd_Even -> Conn_02x20_Odd_Even; footprint Connector_PinHeader_1.27mm:PinHeader_2x21_P1.27mm_Vertical -> Connector_PinHeader_2.54mm:PinHeader_2x20_P2.54mm_Vertical
- J3, J4: footprint Connector_PinHeader_1.27mm:PinHeader_1x08_P1.27mm_Vertical -> Connector_PinHeader_2.54mm:PinHeader_1x08_P2.54mm_Vertical
- J5: footprint Connector_PinHeader_1.27mm:PinHeader_1x03_P1.27mm_Vertical -> Connector_PinHeader_2.54mm:PinHeader_1x03_P2.54mm_Vertical
- J8: footprint Connector_PinHeader_1.27mm:PinHeader_1x05_P1.27mm_Vertical -> Connector_PinHeader_2.54mm:PinHeader_1x05_P2.54mm_Vertical
- J9: footprint Connector_PinHeader_1.27mm:PinHeader_1x08_P1.27mm_Vertical -> Connector_PinHeader_2.54mm:PinHeader_1x05_P2.54mm_Vertical
- RV1: footprint Potentiometer_THT:Potentiometer_Bourns_3296W_Vertical -> 6502Computer:10 kOhms 12 Watt Square Cermet Potentiometer
- U2: value PAL24 -> ATF22V10C
- moved C6 439.8 mm to (366.8, 159.4)
- moved C7 422.5 mm to (376.0, 95.9)
- moved R9 419.9 mm to (351.8, 116.2)
- moved R8 416.4 mm to (351.8, 123.2)
- moved R2 414.5 mm to (352.0, 130.2)
- moved R4 413.6 mm to (351.8, 137.2)
- moved J15 409.5 mm to (312.4, 139.7)
- moved R7 409.1 mm to (326.4, 99.8)
- moved C4 405.1 mm to (330.2, 113.1)
- moved R5 403.7 mm to (298.4, 169.0)
- moved C3 399.8 mm to (320.5, 160.0)
- moved J8 392.2 mm to (343.0, 119.9)
- moved SW2 385.9 mm to (326.9, 85.6)
- moved C16 377.8 mm to (350.5, 87.1), turned to 180 degrees
- moved R1 369.2 mm to (308.6, 99.8)
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Connections:
- J11 pad 2: Net-(J11-Pad2) -> unconnected-(J11-Pad2)
- J11 pad 6: Net-(J11-Pad6) -> unconnected-(J11-Pad6)
- J2 pad 31: EXT_IN2 -> a15
- J2 pad 33: dev4 -> dev7
- J2 pad 35: dev5 -> dev8
- J2 pad 37: dev6 -> dev9
- J2 pad 40: +5V -> GND
- J6 pad 31: EXT_IN2 -> a15
- J6 pad 33: dev7 -> dev10
- J6 pad 35: dev8 -> dev11
- J6 pad 37: dev9 -> dev12
- J6 pad 40: +5V -> GND
- U12 pad 25: EXT_IN2 -> a15
- U12 pad 35: Net-(U12-Pad35) -> unconnected-(U12-Pad35)
- U12 pad 39: Net-(U12-Pad39) -> unconnected-(U12-Pad39)
- U2 pad 3: EXT_IN2 -> a15
- U3 pad 18: EXT_IN2 -> a15
- X1 pad 1: Net-(X1-Pad1) -> unconnected-(X1-Pad1)
Routing:
- net d7: track 0.00 -> 248.1 mm
- net d6: track 0.00 -> 244.5 mm
- net 1pb6: track 0.00 -> 241.5 mm
- net d5: track 0.00 -> 241.1 mm
- net d4: track 0.00 -> 237.4 mm
- net +5V: track 0.00 -> 232.4 mm
- net 1pb5: track 0.00 -> 232.2 mm
- net d3: track 0.00 -> 230.9 mm
- net 1pb4: track 0.00 -> 224.8 mm
- net GND: track 0.00 -> 217.8 mm
- net d0: track 0.00 -> 211.8 mm
- net d1: track 0.00 -> 210.4 mm
- net d2: track 0.00 -> 208.9 mm
- net 1pb0: track 0.00 -> 116.5 mm
- net 1pb1: track 0.00 -> 112.3 mm
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Other:
- board outline added: 274.3 x 185.4 mm
- net class Default removed
- board text added: "Strahinja Marinkovic 6502 Computer"

Commit message: pcb almost done
Parts:
- C12: renamed from C17; footprint Capacitor_THT:C_Disc_D5.1mm_W3.2mm_P5.00mm -> Capacitor_THT:C_Radial_D5.0mm_H11.0mm_P2.00mm
- C13: renamed from C18; footprint Capacitor_THT:C_Disc_D5.1mm_W3.2mm_P5.00mm -> Capacitor_THT:C_Radial_D5.0mm_H11.0mm_P2.00mm
- C6: renamed from C15; footprint Capacitor_THT:C_Radial_D8.0mm_H7.0mm_P3.50mm -> Capacitor_THT:C_Radial_D10.0mm_H20.0mm_P5.00mm
- J5: renamed from J9; footprint Connector_PinHeader_2.54mm:PinHeader_1x05_P2.54mm_Vertical -> Connector_PinHeader_2.54mm:PinHeader_1x08_P2.54mm_Vertical
- moved C7 156.0 mm to (211.5, 145.0)
- moved U3 155.3 mm to (207.1, 159.5)
- moved X1 148.4 mm to (158.4, 191.8)
- moved C8 130.0 mm to (220.5, 91.0), turned to 0 degrees
- moved SW1 107.7 mm to (219.8, 95.8)
- moved R1 107.4 mm to (219.2, 107.0)
- moved SW2 96.1 mm to (219.8, 120.8)
- moved R6 90.5 mm to (219.2, 114.0)
- moved R5 89.3 mm to (274.0, 167.0), turned to 180 degrees
- moved J1 87.7 mm to (280.0, 228.1)
- moved C2 86.3 mm to (297.5, 197.0)
- moved J2 86.0 mm to (280.0, 201.1)
- moved U6 85.5 mm to (292.4, 136.9)
- moved U7 85.5 mm to (292.4, 201.9)
- moved R3 83.8 mm to (274.0, 160.8), turned to 180 degrees
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- renumbered C8 to C10, C9 to C11, C6 to C7, C16 to C8, C7 to C9, J3 to J1, J6 to J10, J7 to J12, J12 to J13, J17 to J14, J4 to J2, J5 to J3, J1 to J4, J8 to J6, J2 to J7, J15 to J8, J13 to J9, R7 to R1, R5 to R2, R2 to R3, R8 to R5, R1 to R6, R9 to R7, R6 to R8, R3 to R9, SW2 to SW1, SW1 to SW2, U13 to U10, U3 to U2, U5 to U3, U2 to U4, U12 to U5, U4 to U6, U10 to U9
Connections:
- J5 pad 1: 1CB1 -> 1CB2
- J5 pad 2: 1CB2 -> 1CB1
Routing:
- net +5V: track 232.4 -> 843.7 mm
- net GND: track 217.8 -> 793.0 mm
- net PHI2: track 66.6 -> 468.3 mm, vias 0 -> 2
- net RW: track 66.5 -> 434.5 mm, vias 0 -> 1
- net a1: track 56.2 -> 387.0 mm
- net a4: track 0.00 -> 328.9 mm
- net a6: track 0.00 -> 324.9 mm, vias 0 -> 1
- net a11: track 0.00 -> 323.1 mm
- net a3: track 56.2 -> 375.4 mm, vias 0 -> 2
- net a2: track 56.2 -> 373.7 mm, vias 0 -> 1
- net a7: track 0.00 -> 314.7 mm, vias 0 -> 1
- net a0: track 56.2 -> 358.9 mm, vias 0 -> 1
- net a10: track 0.00 -> 300.4 mm, vias 0 -> 2
- net a12: track 0.00 -> 299.3 mm, vias 0 -> 1
- net a9: track 0.00 -> 296.2 mm
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Other:
- board size 274.3 x 185.4 mm -> 188.3 x 191.4 mm

Commit message: worked on pcb
Routing:
- net GND: track 793.0 -> 793.7 mm
- net 1CB1: track 73.0 -> 72.3 mm
