File: 6502v2.0/video.kicad_sch (KiCad schematic)
At the start: 7 parts, among them U12 TMS9918A, U16 74LS574, U17 74LS574, U18 74LS574, Y1 Crystal

Commit message: working on video
Connections:
- net d7: now reaches U12.17 (CD7)
- net d6: now reaches U12.18 (CD6)
- net d5: now reaches U12.19 (CD5)
- net d4: now reaches U12.20 (CD4)
- net d3: now reaches U12.21 (CD3)
- net d1: now reaches U12.22 (CD2)
- net d2: now reaches U12.23 (CD1)
- net d0: now reaches U12.24 (CD0)
- net RESET: now reaches U12.34 (RESETB)
Changed lines of the file:
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@@
   (junction (at 53.34 111.76) (diameter 0) (color 0 0 0 0)
   )
+  (bus_entry (at 74.93 78.74) (size 2.54 2.54)
+    (stroke (width 0) (type default))
+  )
+  (bus_entry (at 74.93 71.12) (size 2.54 2.54)
+    (stroke (width 0) (type default))
+  )
+  (bus_entry (at 74.93 68.58) (size 2.54 2.54)
+    (stroke (width 0) (type default))
+  )
+  (bus_entry (at 74.93 76.2) (size 2.54 2.54)
+    (stroke (width 0) (type default))
+  )
+  (bus_entry (at 74.93 66.04) (size 2.54 2.54)
+    (stroke (width 0) (type default))
+  )
+  (bus_entry (at 74.93 73.66) (size 2.54 2.54)
+    (stroke (width 0) (type default))
+  )
+  (bus_entry (at 74.93 81.28) (size 2.54 2.54)
+    (stroke (width 0) (type default))
+  )
+  (bus_entry (at 74.93 63.5) (size 2.54 2.54)
+    (stroke (width 0) (type default))
+  )
   (wire (pts (xy 67.31 99.06) (xy 82.55 99.06))
     (stroke (width 0) (type default))
   )
+  (bus (pts (xy 74.93 63.5) (xy 74.93 66.04))
+    (stroke (width 0) (type default))
+  )
+  (wire (pts (xy 77.47 76.2) (xy 82.55 76.2))
+    (stroke (width 0) (type default))
+  )
   (wire (pts (xy 60.96 97.79) (xy 67.31 97.79))
     (stroke (width 0) (type default))
   )
+  (wire (pts (xy 77.47 73.66) (xy 82.55 73.66))
+    (stroke (width 0) (type default))
+  )
+  (wire (pts (xy 77.47 81.28) (xy 82.55 81.28))
+    (stroke (width 0) (type default))
+  )
+  (wire (pts (xy 77.47 68.58) (xy 82.55 68.58))
+    (stroke (width 0) (type default))
+  )
+  (wire (pts (xy 77.47 71.12) (xy 82.55 71.12))
+    (stroke (width 0) (type default))
+  )
+  (bus (pts (xy 74.93 66.04) (xy 74.93 68.58))
+    (stroke (width 0) (type default))
+  )
+  (wire (pts (xy 77.47 83.82) (xy 82.55 83.82))
+    (stroke (width 0) (type default))
+  )
   (wire (pts (xy 67.31 111.76) (xy 67.31 106.68))
     (stroke (width 0) (type default))
@@
     (stroke (width 0) (type default))
   )
+  (bus (pts (xy 74.93 73.66) (xy 74.93 76.2))
+    (stroke (width 0) (type default))
+  )
   (wire (pts (xy 60.96 111.76) (xy 67.31 111.76))
     (stroke (width 0) (type default))
   )
+  (bus (pts (xy 74.93 71.12) (xy 74.93 73.66))
+    (stroke (width 0) (type default))
+  )
   (wire (pts (xy 82.55 106.68) (xy 82.55 102.87))
     (stroke (width 0) (type default))
   )
+  (bus (pts (xy 74.93 68.58) (xy 74.93 71.12))
+    (stroke (width 0) (type default))
+  )
+  (bus (pts (xy 74.93 78.74) (xy 74.93 81.28))
+    (stroke (width 0) (type default))
+  )
+  (wire (pts (xy 77.47 66.04) (xy 82.55 66.04))
+    (stroke (width 0) (type default))
+  )
+  (wire (pts (xy 77.47 78.74) (xy 82.55 78.74))
+    (stroke (width 0) (type default))
+  )
   (wire (pts (xy 67.31 97.79) (xy 67.31 99.06))
     (stroke (width 0) (type default))
   )
+  (bus (pts (xy 74.93 76.2) (xy 74.93 78.74))
+    (stroke (width 0) (type default))
+  )
   (wire (pts (xy 82.55 99.06) (xy 82.55 100.33))
     (stroke (width 0) (type default))
@@
   (wire (pts (xy 67.31 106.68) (xy 82.55 106.68))
     (stroke (width 0) (type default))
+  )
+  (label "d6" (at 80.01 81.28 0) (fields_autoplaced)
+    (effects (font (size 1.27 1.27)) (justify left bottom))
+  )
+  (label "d4" (at 80.01 76.2 0) (fields_autoplaced)
+    (effects (font (size 1.27 1.27)) (justify left bottom))
+  )
+  (label "d1" (at 80.01 68.58 0) (fields_autoplaced)
+    (effects (font (size 1.27 1.27)) (justify left bottom))
+  )
+  (label "d3" (at 80.01 73.66 0) (fields_autoplaced)
+    (effects (font (size 1.27 1.27)) (justify left bottom))
+  )
+  (label "d5" (at 80.01 78.74 0) (fields_autoplaced)
+    (effects (font (size 1.27 1.27)) (justify left bottom))
+  )
+  (label "d0" (at 80.01 66.04 0) (fields_autoplaced)
+    (effects (font (size 1.27 1.27)) (justify left bottom))
+  )
+  (label "d7" (at 80.01 83.82 0) (fields_autoplaced)
+    (effects (font (size 1.27 1.27)) (justify left bottom))
+  )
+  (label "d2" (at 80.01 71.12 0) (fields_autoplaced)
+    (effects (font (size 1.27 1.27)) (justify left bottom))
+  )
+  (global_label "RESET" (shape input) (at 82.55 97.79 180) (fields_autoplaced)
+    (effects (font (size 1.27 1.27)) (justify right))
+    (property "Intersheetrefs" "${INTERSHEET_REFS}" (at 73.8991 97.79 0)
+      (effects (font (size 1.27 1.27)) (justify right) hide)
+    )
+  )
+  (global_label "d[0..7]" (shape input) (at 74.93 81.28 180) (fields_autoplaced)
+    (effects (font (size 1.27 1.27)) (justify right))
+    (property "Intersheetrefs" "${INTERSHEET_REFS}" (at 65.5532 81.28 0)
+      (effects (font (size 1.27 1.27)) (justify right) hide)
+    )
   )
   (symbol (lib_id "power:+5V") (at 160.02 120.65 0) (unit 1)
@@
     )
   )
+  (symbol (lib_id "Device:Crystal") (at 67.31 102.87 270) (unit 1)
+    (in_bom yes) (on_board yes) (dnp no) (fields_autoplaced)
+    (property "Reference" "Y1" (at 71.12 101.6 90)
+      (effects (font (size 1.27 1.27)) (justify left))
+    )
+    (property "Value" "Crystal" (at 71.12 104.14 90)
+      (effects (font (size 1.27 1.27)) (justify left))
+    )
+    (property "Footprint" "" (at 67.31 102.87 0)
+      (effects (font (size 1.27 1.27)) hide)
+    )
+    (property "Datasheet" "~" (at 67.31 102.87 0)
+      (effects (font (size 1.27 1.27)) hide)
+    )
+    (pin "1")
+    (pin "2")
+    (instances
+      (project "6502v2.0"
+        (path "/5ffbcd12-d35a-40f1-aa31-5cc41b65e9d8/44a321ed-5b62-41df-a171-68eb6641f1e1"
+          (reference "Y1") (unit 1)
+        )
+      )
+    )
+  )
   (symbol (lib_id "GraphicsLibrary:TMS9918A") (at 91.44 83.82 0) (unit 1)
     (in_bom yes) (on_board yes) (dnp no) (fields_autoplaced)
-    (property "Reference" "U12" (at 93.3959 55.88 0)
-      (effects (font (size 1.27 1.27)) (justify left))
-    )
-    (property "Value" "TMS9918A" (at 93.3959 58.42 0)
+    (property "Reference" "U12" (at 93.3959 57.15 0)
+      (effects (font (size 1.27 1.27)) (justify left))
+    )
+    (property "Value" "TMS9918A" (at 93.3959 59.69 0)
       (effects (font (size 1.27 1.27)) (justify left))
     )
@@
         )
       )
-    )
-  )
-  (symbol (lib_id "Device:Crystal") (at 67.31 102.87 270) (unit 1)
-    (in_bom yes) (on_board yes) (dnp no) (fields_autoplaced)
-    (property "Reference" "Y1" (at 71.12 101.6 90)
-      (effects (font (size 1.27 1.27)) (justify left))
-    )
-    (property "Value" "Crystal" (at 71.12 104.14 90)
-      (effects (font (size 1.27 1.27)) (justify left))
-    )
-    (property "Footprint" "" (at 67.31 102.87 0)
-      (effects (font (size 1.27 1.27)) hide)
-    )
-    (property "Datasheet" "~" (at 67.31 102.87 0)
-      (effects (font (size 1.27 1.27)) hide)
-    )
-    (pin "1")
-    (pin "2")
-    (instances
-      (project "6502v2.0"
-        (path "/5ffbcd12-d35a-40f1-aa31-5cc41b65e9d8/44a321ed-5b62-41df-a171-68eb6641f1e1"
-          (reference "Y1") (unit 1)
-        )
-      )

Commit message: working on pcb
Parts:
- added C23: 0.1uF, Capacitor_THT:C_Disc_D5.1mm_W3.2mm_P5.00mm, symbol Device:C
- added FB1: FerriteBead, symbol Device:FerriteBead
- added J17: Conn_Coaxial, symbol Connector:Conn_Coaxial
- added Q3: NPN, symbol Simulation_SPICE:NPN
- added R26: 470, Resistor_THT:R_Axial_DIN0204_L3.6mm_D1.6mm_P7.62mm_Horizontal, symbol Device:R
- added R27: 75, Resistor_THT:R_Axial_DIN0204_L3.6mm_D1.6mm_P7.62mm_Horizontal, symbol Device:R
- added U19: HM62256BLP, Package_DIP:DIP-28_W15.24mm, symbol Memory_RAM:HM62256BLP
- C21, C22: footprint (none) -> Capacitor_THT:C_Disc_D5.1mm_W3.2mm_P5.00mm
- U12: footprint (none) -> Package_DIP:DIP-40_W15.24mm_Socket
- U16, U17, U18: footprint (none) -> Package_DIP:DIP-20_W7.62mm_Socket
Connections:
- net +5V: now also FB1.2, U19.28 (VCC)
- net GND: now also C23.1, J17.2 (Ext), R26.2, R27.2, U19.14 (GND)
- net VA0: now reaches U16.2 (D0)
- net VA0: now also U12.10 (AD0), U17.2 (D0), U18.2 (D0)
- net VA1: now reaches U16.3 (D1)
- net VA1: now also U12.9 (AD1), U17.3 (D1), U18.3 (D1)
- net VA2: now reaches U16.4 (D2)
- net VA2: now also U12.8 (AD2), U17.4 (D2), U18.4 (D2)
- net VA3: now reaches U16.5 (D3)
- net VA3: now also U12.7 (AD3), U17.5 (D3), U18.5 (D3)
- net VA4: now reaches U16.6 (D4)
- net VA4: now also U12.6 (AD4), U17.6 (D4), U18.6 (D4)
- net VA5: now reaches U16.7 (D5)
- net VA5: now also U12.5 (AD5), U17.7 (D5), U18.7 (D5)
- net VA6: now reaches U16.8 (D6)
- net VA6: now also U12.4 (AD6), U17.8 (D6), U18.8 (D6)
- net VA7: now reaches U16.9 (D7)
- net VA7: now also U12.3 (AD7), U17.9 (D7), U18.9 (D7)
- net at U12.36 (COMVID): now also Q3.2 (B), R26.1
- new net: C23.2, FB1.1, Q3.1 (C)
- new net: J17.1 (In), Q3.3 (E), R27.1
Other:
- moved on the sheet: U16, U17, U18

Commit message: trying new compiler
Parts:
- added U20: 74HC04, symbol 74xx:74HC04
Other:
- moved on the sheet: U19

Commit message: worked on video card
Parts:
- U12: footprint Package_DIP:DIP-40_W15.24mm_Socket -> (none)
Connections:
- net +5V: now also U20.14 (VCC)
- net GND: now also U16.1 (OE), U17.1 (OE), U18.1 (OE), U20.7 (GND)
- net RAS: now reaches U12.1 (RASB)
- net RAS: now also U20.5
- net VRW: now reaches U12.11 (RWB)
- net VRW: now also U19.27 (~{WE}), U20.1
- net CAS: now reaches U12.2 (CASB)
- net CAS: now also U19.20 (~{CS}), U20.9
- net RD7: now reaches U12.25 (RD7)
- net RD7: now also U16.12 (Q7), U19.19 (Q7)
- net RD6: now reaches U12.26 (RD6)
- net RD6: now also U16.13 (Q6), U19.18 (Q6)
- net RD5: now reaches U12.27 (RD5)
- net RD5: now also U16.14 (Q5), U19.17 (Q5)
- net RD4: now reaches U12.28 (RD4)
- net RD4: now also U16.15 (Q4), U19.16 (Q4)
- net RD3: now reaches U12.29 (RD3)
- net RD3: now also U16.16 (Q3), U19.15 (Q3)
- net RD2: now reaches U12.30 (RD2)
- net RD2: now also U16.17 (Q2), U19.13 (Q2)
- net RD1: now reaches U12.31 (RD1)
- net RD1: now also U16.18 (Q1), U19.12 (Q1)
- net RD0: now reaches U12.32 (RD0)
- net RD0: now also U16.19 (Q0), U19.11 (Q0)
- net ROW: now reaches U18.11 (Cp)
- net ROW: now also U20.6
- net at U18.12 (Q7): now also U19.4 (A6)
- net at U18.13 (Q6): now also U19.5 (A5)
- net at U18.14 (Q5): now also U19.6 (A4)
- net at U18.15 (Q4): now also U19.7 (A3)
- net at U18.16 (Q3): now also U19.8 (A2)
- net at U18.17 (Q2): now also U19.9 (A1)
- net at U18.18 (Q1): now also U19.10 (A0)
- net at U19.1 (A14): now also U17.12 (Q7), U19.26 (A13)
- net at U19.2 (A12): now also U17.13 (Q6)
- net at U19.21 (A10): now also U17.15 (Q4)
- net VWR: now reaches U19.22 (~{OE})
- net VWR: now also U20.2, U20.3
- net at U19.23 (A11): now also U17.14 (Q5)
- net at U19.24 (A9): now also U17.16 (Q3)
- net at U19.25 (A8): now also U17.17 (Q2)
- net at U19.3 (A7): now also U17.18 (Q1)
- net COL: now reaches U17.11 (Cp)
- net COL: now also U20.12
- net at U20.8: now also U20.11
- net VRD: now reaches U20.4
- net at U20.13: now also U20.10
- no-connect marks 0 -> 2
Other:
- moved on the sheet: C21, C22, C23, FB1, J17, Q3, R26, R27, U19, U20A, U20B, U20C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

Commit message: changes
Parts:
- added U21: 74LS138, symbol 74xx:74LS138
Connections:
- net +5V: now also U21.16 (VCC), U21.6 (E3)
- net GND: now also U21.2 (A1), U21.3 (A2), U21.8 (GND)
- net a0: now reaches U12.13 (MODE)
- net at U12.14 (CSWB): now also U21.15 (O0)
- net at U12.15 (CSRB): now also U21.14 (O1)
- new net RW: U21.1 (A0)
- new net VDP_CS: U21.4 (E1), U21.5 (E2)
- no-connect marks 2 -> 8
Other:
- moved on the sheet: C21, C22, C23, FB1, J17, Q3, R26, R27, U12, Y1
