File: 6502v2.0/audio.kicad_sch (KiCad schematic)
At the start: 15 parts, among them U13 PSG_AY-3-8910, U15 PSG_AY-3-8910

Commit message: worked on sound stuff
Parts:
- added J1 (x2): ~, symbol Connector_Generic:Conn_01x08
Connections:
- net +5V: now also R14.1
- net 2pa7: now reaches U13.30 (D7)
- net 2pa6: now reaches U13.31 (D6)
- net 2pa5: now reaches U13.32 (D5)
- net 2pa4: now reaches U13.33 (D4)
- net 2pa3: now reaches U13.34 (D3)
- net 2pa2: now reaches U13.35 (D2)
- net 2pa1: now reaches U13.36 (D1)
- net 2pa0: now reaches U13.37 (D0)
- net PSG2IOB3: now reaches U15.10 (IOB3)
- net PSG2IOB3: now also J1.5 (Pin_5)
- net PSG2IOB2: now reaches U15.11 (IOB2)
- net PSG2IOB2: now also J1.6 (Pin_6)
- net PSG2IOB1: now reaches U15.12 (IOB1)
- net PSG2IOB1: now also J1.7 (Pin_7)
- net PSG2IOB0: now reaches U15.13 (IOB0)
- net PSG2IOB0: now also J1.8 (Pin_8)
- net PSGIOA7: now reaches U15.14 (IOA7)
- net PSGIOA7: now also J1.1 (Pin_1)
- net PSGIOA6: now reaches U15.15 (IOA6)
- net PSGIOA6: now also J1.2 (Pin_2)
- net PSGIOA5: now reaches U15.16 (IOA5)
- net PSGIOA5: now also J1.3 (Pin_3)
- net PSGIOA4: now reaches U15.17 (IOA4)
- net PSGIOA4: now also J1.4 (Pin_4)
- net PSGIOA3: now reaches U15.18 (IOA3)
- net PSGIOA3: now also J1.5 (Pin_5)
- net PSGIOA2: now reaches U15.19 (IOA2)
- net PSGIOA2: now also J1.6 (Pin_6)
- net PSGIOA1: now reaches U15.20 (IOA1)
- net PSGIOA1: now also J1.7 (Pin_7)
- net PSGIOA0: now reaches U15.21 (IOA0)
- net PSGIOA0: now also J1.8 (Pin_8)
- net PSG2IOB7: now reaches U15.6 (IOB7)
- net PSG2IOB7: now also J1.1 (Pin_1)
- net PSG2IOB6: now reaches U15.7 (IOB6)
- net PSG2IOB6: now also J1.2 (Pin_2)
- net PSG2IOB5: now reaches U15.8 (IOB5)
- net PSG2IOB5: now also J1.3 (Pin_3)
- net PSG2IOB4: now reaches U15.9 (IOB4)
- net PSG2IOB4: now also J1.4 (Pin_4)

Commit message: stuff
Parts:
- added J1: ~, symbol Connector_Generic:Conn_01x08
- added J16: AudioPlug3, symbol Connector_Audio:AudioPlug3
- added R23, R24, R25: 1K, symbol Device:R
Connections:
- net +5V: now also R25.1; no longer U15.28 (BC2)
- net AUDIO_OUT_LEFT: now also J16.T
- net AUDIO_OUT_RIGHT: now also J16.R
- net GND: now also J16.S, R23.2, R24.2; no longer U15.24 (~{A9})
- net PSG2IOB0: now also J1.1 (Pin_1); no longer J1.8 (Pin_8)
- net PSG2IOB1: now also J1.2 (Pin_2); no longer J1.7 (Pin_7)
- net PSG2IOB2: now also J1.3 (Pin_3); no longer J1.6 (Pin_6)
- net PSG2IOB3: now also J1.4 (Pin_4); no longer J1.5 (Pin_5)
- net PSG2IOB4: now also J1.5 (Pin_5); no longer J1.4 (Pin_4)
- net PSG2IOB5: now also J1.6 (Pin_6); no longer J1.3 (Pin_3)
- net PSG2IOB6: now also J1.7 (Pin_7); no longer J1.2 (Pin_2)
- net PSG2IOB7: now also J1.8 (Pin_8); no longer J1.1 (Pin_1)
- net PSGIOA0: now also J1.1 (Pin_1); no longer J1.8 (Pin_8)
- net PSGIOA1: now also J1.2 (Pin_2); no longer J1.7 (Pin_7)
- net PSGIOA2: now also J1.3 (Pin_3); no longer J1.6 (Pin_6)
- net PSGIOA3: now also J1.4 (Pin_4); no longer J1.5 (Pin_5)
- net PSGIOA4: now also J1.5 (Pin_5); no longer J1.4 (Pin_4)
- net PSGIOA5: now also J1.6 (Pin_6); no longer J1.3 (Pin_3)
- net PSGIOA6: now also J1.7 (Pin_7); no longer J1.2 (Pin_2)
- net PSGIOA7: now also J1.8 (Pin_8); no longer J1.1 (Pin_1)
- net at R14.2, U15.25 (A8): now also U15.28 (BC2)
- net PSG1IOB3: now reaches U13.10 (IOB3)
- net PSG1IOB3: now also J1.4 (Pin_4)
- net PSG1IOB2: now reaches U13.11 (IOB2)
- net PSG1IOB2: now also J1.3 (Pin_3)
- net at U13.24 (~{A9}): now also R24.1
- net at U13.25 (A8): now also U13.28 (BC2), R25.2
- net 1pa7: now reaches U13.27 (BDIR)
- net 1pa6: now reaches U13.29 (BC1)
- net PSG1IOB7: now reaches U13.6 (IOB7)
- net PSG1IOB7: now also J1.8 (Pin_8)
- net PSG1IOB6: now reaches U13.7 (IOB6)
- net PSG1IOB6: now also J1.7 (Pin_7)
- net PSG1IOB5: now reaches U13.8 (IOB5)
- net PSG1IOB5: now also J1.6 (Pin_6)
- net PSG1IOB4: now reaches U13.9 (IOB4)
- net PSG1IOB4: now also J1.5 (Pin_5)
- new net: R23.1, U15.24 (~{A9})
- no-connect marks 4 -> 6
Other:
- moved on the sheet: J1

Commit message: working on pcb
Parts:
- C16, C18, C19, C20: footprint (none) -> Capacitor_THT:C_Disc_D5.1mm_W3.2mm_P5.00mm
- R14, R15, R16, R17, R18, R19, R20, R21, R22, R23, R24, R25: footprint (none) -> Resistor_THT:R_Axial_DIN0204_L3.6mm_D1.6mm_P7.62mm_Horizontal
- U13, U15: footprint (none) -> Package_DIP:DIP-40_W15.24mm_Socket
Changed lines of the file:
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@@
       (effects (font (size 1.27 1.27)) (justify left))
     )
-    (property "Footprint" "" (at 113.792 45.72 90)
+    (property "Footprint" "Resistor_THT:R_Axial_DIN0204_L3.6mm_D1.6mm_P7.62mm_Horizontal" (at 113.792 45.72 90)
       (effects (font (size 1.27 1.27)) hide)
     )
@@
       (effects (font (size 1.27 1.27)) (justify left))
     )
-    (property "Footprint" "" (at 113.792 102.87 90)
+    (property "Footprint" "Resistor_THT:R_Axial_DIN0204_L3.6mm_D1.6mm_P7.62mm_Horizontal" (at 113.792 102.87 90)
       (effects (font (size 1.27 1.27)) hide)
     )
@@
       (effects (font (size 1.27 1.27)) (justify right))
     )
-    (property "Footprint" "" (at 85.598 114.3 90)
+    (property "Footprint" "Resistor_THT:R_Axial_DIN0204_L3.6mm_D1.6mm_P7.62mm_Horizontal" (at 85.598 114.3 90)
       (effects (font (size 1.27 1.27)) hide)
     )
@@
       (effects (font (size 1.27 1.27)) (justify right))
     )
-    (property "Footprint" "" (at 184.658 69.85 90)
+    (property "Footprint" "Resistor_THT:R_Axial_DIN0204_L3.6mm_D1.6mm_P7.62mm_Horizontal" (at 184.658 69.85 90)
       (effects (font (size 1.27 1.27)) hide)
     )
@@
       (effects (font (size 1.27 1.27)) (justify left))
     )
-    (property "Footprint" "" (at 189.992 77.47 90)
+    (property "Footprint" "Resistor_THT:R_Axial_DIN0204_L3.6mm_D1.6mm_P7.62mm_Horizontal" (at 189.992 77.47 90)
       (effects (font (size 1.27 1.27)) hide)
     )
@@
       (effects (font (size 1.27 1.27)) (justify left))
     )
-    (property "Footprint" "" (at 82.042 121.92 90)
+    (property "Footprint" "Resistor_THT:R_Axial_DIN0204_L3.6mm_D1.6mm_P7.62mm_Horizontal" (at 82.042 121.92 90)
       (effects (font (size 1.27 1.27)) hide)
     )
@@
       (effects (font (size 1.27 1.27)) (justify right))
     )
-    (property "Footprint" "" (at 94.488 114.3 90)
+    (property "Footprint" "Resistor_THT:R_Axial_DIN0204_L3.6mm_D1.6mm_P7.62mm_Horizontal" (at 94.488 114.3 90)
       (effects (font (size 1.27 1.27)) hide)
     )
@@
       (effects (font (size 1.27 1.27)) (justify left))
     )
-    (property "Footprint" "" (at 16.002 36.83 90)
+    (property "Footprint" "Resistor_THT:R_Axial_DIN0204_L3.6mm_D1.6mm_P7.62mm_Horizontal" (at 16.002 36.83 90)
       (effects (font (size 1.27 1.27)) hide)
     )
@@
       (effects (font (size 1.27 1.27)) (justify left))
     )
-    (property "Footprint" "" (at 210.5152 92.71 0)
+    (property "Footprint" "Capacitor_THT:C_Disc_D5.1mm_W3.2mm_P5.00mm" (at 210.5152 92.71 0)
       (effects (font (size 1.27 1.27)) hide)
     )
@@
       (effects (font (size 1.27 1.27)) (justify left))
     )
-    (property "Footprint" "" (at 26.162 95.25 90)
+    (property "Footprint" "Resistor_THT:R_Axial_DIN0204_L3.6mm_D1.6mm_P7.62mm_Horizontal" (at 26.162 95.25 90)
       (effects (font (size 1.27 1.27)) hide)
     )
@@
       (effects (font (size 1.27 1.27)))
     )
-    (property "Footprint" "" (at 217.17 72.6948 0)
+    (property "Footprint" "Capacitor_THT:C_Disc_D5.1mm_W3.2mm_P5.00mm" (at 217.17 72.6948 0)
       (effects (font (size 1.27 1.27)) hide)
     )
@@
       (effects (font (size 1.27 1.27)) (justify right))
     )
-    (property "Footprint" "" (at 193.548 69.85 90)
+    (property "Footprint" "Resistor_THT:R_Axial_DIN0204_L3.6mm_D1.6mm_P7.62mm_Horizontal" (at 193.548 69.85 90)
       (effects (font (size 1.27 1.27)) hide)
     )
@@
       (effects (font (size 1.27 1.27)) (justify left))
     )
-    (property "Footprint" "" (at 102.5652 137.16 0)
+    (property "Footprint" "Capacitor_THT:C_Disc_D5.1mm_W3.2mm_P5.00mm" (at 102.5652 137.16 0)
       (effects (font (size 1.27 1.27)) hide)
     )
@@
       (effects (font (size 1.27 1.27)))
     )
-    (property "Footprint" "" (at 109.22 117.1448 0)
+    (property "Footprint" "Capacitor_THT:C_Disc_D5.1mm_W3.2mm_P5.00mm" (at 109.22 117.1448 0)
       (effects (font (size 1.27 1.27)) hide)
     )
@@
       (effects (font (size 1.27 1.27)) (justify right))
     )
-    (property "Footprint" "" (at 202.438 69.85 90)
+    (property "Footprint" "Resistor_THT:R_Axial_DIN0204_L3.6mm_D1.6mm_P7.62mm_Horizontal" (at 202.438 69.85 90)
       (effects (font (size 1.27 1.27)) hide)
     )
@@
       (effects (font (size 1.27 1.27)) (justify left))
     )
-    (property "Footprint" "" (at 58.42 34.29 0)
+    (property "Footprint" "Package_DIP:DIP-40_W15.24mm_Socket" (at 58.42 34.29 0)
       (effects (font (size 1.27 1.27)) hide)
     )
@@
       (effects (font (size 1.27 1.27)) (justify left))
     )
-    (property "Footprint" "" (at 142.24 50.8 0)
+    (property "Footprint" "Package_DIP:DIP-40_W15.24mm_Socket" (at 142.24 50.8 0)
       (effects (font (size 1.27 1.27)) hide)
     )
@@
       (effects (font (size 1.27 1.27)) (justify right))
     )
-    (property "Footprint" "" (at 76.708 114.3 90)
-      (effects (font (size 1.27 1.27)) hide)
-    )
+    (property "Footprint" "Resistor_THT:R_Axial_DIN0204_L3.6mm_D1.6mm_P7.62mm_Horizontal" (at 76.708 114.3 90)
+      (effects (font (size 1.27 1.27)) hide)
+    )

Commit message: worked on video card
Other:
- moved on the sheet: J1

Commit message: changes
Connections:
- net +5V: now also U13.28 (BC2), U15.28 (BC2)
- net at R14.2, U15.25 (A8): no longer U15.28 (BC2)
- net at R25.2, U13.25 (A8): no longer U13.28 (BC2)
Changed lines of the file:
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@@
   (junction (at 83.82 118.11) (diameter 0) (color 0 0 0 0)
-  )
-  (junction (at 124.46 85.09) (diameter 0) (color 0 0 0 0)
-  )
-  (junction (at 17.78 63.5) (diameter 0) (color 0 0 0 0)
   )
   (junction (at 191.77 73.66) (diameter 0) (color 0 0 0 0)
@@
     (stroke (width 0) (type default))
   )
-  (wire (pts (xy 17.78 63.5) (xy 17.78 40.64))
-    (stroke (width 0) (type default))
-  )
   (wire (pts (xy 264.16 93.98) (xy 255.27 93.98))
     (stroke (width 0) (type default))
@@
     (stroke (width 0) (type default))
   )
-  (wire (pts (xy 17.78 68.58) (xy 17.78 63.5))
+  (wire (pts (xy 17.78 40.64) (xy 17.78 68.58))
     (stroke (width 0) (type default))
   )
@@
     (stroke (width 0) (type default))
   )
-  (wire (pts (xy 124.46 80.01) (xy 124.46 85.09))
-    (stroke (width 0) (type default))
-  )
   (bus (pts (xy 162.56 83.82) (xy 162.56 86.36))
     (stroke (width 0) (type default))
@@
     (stroke (width 0) (type default))
   )
-  (wire (pts (xy 17.78 63.5) (xy 39.37 63.5))
-    (stroke (width 0) (type default))
-  )
   (wire (pts (xy 264.16 116.84) (xy 256.54 116.84))
     (stroke (width 0) (type default))
@@
     (stroke (width 0) (type default))
   )
+  (wire (pts (xy 25.4 62.23) (xy 46.99 62.23))
+    (stroke (width 0) (type default))
+  )
   (bus (pts (xy 163.83 101.6) (xy 163.83 104.14))
     (stroke (width 0) (type default))
@@
     (stroke (width 0) (type default))
   )
+  (wire (pts (xy 124.46 41.91) (xy 124.46 80.01))
+    (stroke (width 0) (type default))
+  )
   (wire (pts (xy 200.66 55.88) (xy 200.66 66.04))
     (stroke (width 0) (type default))
@@
     (stroke (width 0) (type default))
   )
-  (wire (pts (xy 115.57 85.09) (xy 124.46 85.09))
-    (stroke (width 0) (type default))
-  )
   (bus (pts (xy 162.56 88.9) (xy 162.56 91.44))
     (stroke (width 0) (type default))
   )
+  (wire (pts (xy 25.4 33.02) (xy 25.4 62.23))
+    (stroke (width 0) (type default))
+  )
   (wire (pts (xy 83.82 44.45) (xy 68.58 44.45))
     (stroke (width 0) (type default))
@@
     (stroke (width 0) (type default))
   )
+  (wire (pts (xy 46.99 62.23) (xy 46.99 63.5))
+    (stroke (width 0) (type default))
+  )
   (wire (pts (xy 182.88 73.66) (xy 191.77 73.66))
     (stroke (width 0) (type default))
@@
     (stroke (width 0) (type default))
   )
-  (wire (pts (xy 39.37 63.5) (xy 46.99 63.5))
-    (stroke (width 0) (type default))
-  )
   (wire (pts (xy 118.11 82.55) (xy 130.81 82.55))
     (stroke (width 0) (type default))
@@
     (stroke (width 0) (type default))
   )
-  (wire (pts (xy 124.46 85.09) (xy 130.81 85.09))
+  (wire (pts (xy 115.57 85.09) (xy 130.81 85.09))
     (stroke (width 0) (type default))
   )
@@
         (path "/5ffbcd12-d35a-40f1-aa31-5cc41b65e9d8/99446e73-4cf8-4cf8-b0e5-2db38fecee4d"
           (reference "R23") (unit 1)
+        )
+      )
+    )
+  )
+  (symbol (lib_id "power:+5V") (at 124.46 41.91 0) (unit 1)
+    (in_bom yes) (on_board yes) (dnp no) (fields_autoplaced)
+    (property "Reference" "#PWR0110" (at 124.46 45.72 0)
+      (effects (font (size 1.27 1.27)) hide)
+    )
+    (property "Value" "+5V" (at 124.46 36.83 0)
+      (effects (font (size 1.27 1.27)))
+    )
+    (property "Footprint" "" (at 124.46 41.91 0)
+      (effects (font (size 1.27 1.27)) hide)
+    )
+    (property "Datasheet" "" (at 124.46 41.91 0)
+      (effects (font (size 1.27 1.27)) hide)
+    )
+    (pin "1")
+    (instances
+      (project "6502v2.0"
+        (path "/5ffbcd12-d35a-40f1-aa31-5cc41b65e9d8/99446e73-4cf8-4cf8-b0e5-2db38fecee4d"
+          (reference "#PWR0110") (unit 1)
         )
       )
@@
         )
       )
+    )
+  )
+  (symbol (lib_id "power:+5V") (at 25.4 33.02 0) (unit 1)
+    (in_bom yes) (on_board yes) (dnp no) (fields_autoplaced)
+    (property "Reference" "#PWR0111" (at 25.4 36.83 0)
+      (effects (font (size 1.27 1.27)) hide)
+    )
+    (property "Value" "+5V" (at 25.4 27.94 0)
+      (effects (font (size 1.27 1.27)))
+    )
+    (property "Footprint" "" (at 25.4 33.02 0)
+      (effects (font (size 1.27 1.27)) hide)
+    )
+    (property "Datasheet" "" (at 25.4 33.02 0)
+      (effects (font (size 1.27 1.27)) hide)
+    )
+    (pin "1")
+    (instances
+      (project "6502v2.0"
+        (path "/5ffbcd12-d35a-40f1-aa31-5cc41b65e9d8/99446e73-4cf8-4cf8-b0e5-2db38fecee4d"
+          (reference "#PWR0111") (unit 1)
+        )
+      )
