File: 6502v2.0/audio.kicad_sch (KiCad schematic)
At the start: 27 parts, among them J17 SJ1-2503A, U13 7402, U14 PSG_AY-3-8910, U15 PSG_AY-3-8910

Commit message: working on pcb
Parts:
- removed J17: SJ1-2503A, symbol SJ1-2503A:SJ1-2503A
- added J18: 35RAPC4BV4, 8bits:SWITCHCRAFT_35RAPC4BV4, symbol 35RAPC4BV4:35RAPC4BV4
- C21: renamed from C20; footprint Capacitor_THT:C_Disc_D5.1mm_W3.2mm_P5.00mm -> Capacitor_THT:C_Radial_D5.0mm_H11.0mm_P2.00mm
- C26: renamed from C25; footprint Capacitor_THT:C_Disc_D5.1mm_W3.2mm_P5.00mm -> Capacitor_THT:C_Radial_D5.0mm_H11.0mm_P2.00mm
- renumbered C21 to C22, C26 to C27
Connections:
- net AUDIO_OUT_LEFT: now also J18.2
- net AUDIO_OUT_RIGHT: now also J18.4
- net GND: now also J18.1
- no-connect marks 5 -> 6

Commit message: trying to get basic to work
Parts:
- renumbered C21 to C22, C22 to C23, C26 to C27, C27 to C28, R15 to R13, R16 to R14, R17 to R15, R18 to R16, R19 to R17, R20 to R18, R21 to R19, R22 to R20, R23 to R21, R24 to R22, R25 to R23, R26 to R24, U13 to U14, U14 to U15, U15 to U16

Commit message: redid pcb
Parts:
- renumbered J18 to J19
Changed lines of the file:
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@@
         )
         (path "/5ffbcd12-d35a-40f1-aa31-5cc41b65e9d8/99446e73-4cf8-4cf8-b0e5-2db38fecee4d"
-          (reference "J14") (unit 1)
+          (reference "J15") (unit 1)
         )
       )
@@
   (symbol (lib_id "35RAPC4BV4:35RAPC4BV4") (at 161.29 137.16 0) (unit 1)
     (in_bom yes) (on_board yes) (dnp no) (fields_autoplaced)
-    (property "Reference" "J18" (at 160.776 127 0)
+    (property "Reference" "J19" (at 160.776 127 0)
       (effects (font (size 1.27 1.27)))
     )
@@
       (project "6502v2.0"
         (path "/5ffbcd12-d35a-40f1-aa31-5cc41b65e9d8/99446e73-4cf8-4cf8-b0e5-2db38fecee4d"
-          (reference "J18") (unit 1)
+          (reference "J19") (unit 1)
         )
       )
@@
         )
         (path "/5ffbcd12-d35a-40f1-aa31-5cc41b65e9d8/99446e73-4cf8-4cf8-b0e5-2db38fecee4d"
-          (reference "J15") (unit 1)
+          (reference "J16") (unit 1)
         )
       )
@@
         )
         (path "/5ffbcd12-d35a-40f1-aa31-5cc41b65e9d8/99446e73-4cf8-4cf8-b0e5-2db38fecee4d"
-          (reference "J17") (unit 1)
+          (reference "J18") (unit 1)
         )
       )
@@
         )
         (path "/5ffbcd12-d35a-40f1-aa31-5cc41b65e9d8/99446e73-4cf8-4cf8-b0e5-2db38fecee4d"
-          (reference "J16") (unit 1)
-        )
-      )
+          (reference "J17") (unit 1)
+        )
+      )

Commit message: pcb
Parts:
- C22, C27: footprint Capacitor_THT:C_Radial_D5.0mm_H11.0mm_P2.00mm -> Capacitor_THT:CP_Radial_Tantal_D5.0mm_P2.50mm
Changed lines of the file:
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@@
       (effects (font (size 1.27 1.27)) (justify left))
     )
-    (property "Footprint" "Capacitor_THT:C_Radial_D5.0mm_H11.0mm_P2.00mm" (at 268.9352 91.44 0)
+    (property "Footprint" "Capacitor_THT:CP_Radial_Tantal_D5.0mm_P2.50mm" (at 268.9352 91.44 0)
       (effects (font (size 1.27 1.27)) hide)
     )
@@
       (effects (font (size 1.27 1.27)) (justify left))
     )
-    (property "Footprint" "Capacitor_THT:C_Radial_D5.0mm_H11.0mm_P2.00mm" (at 136.8552 137.16 0)
-      (effects (font (size 1.27 1.27)) hide)
-    )
+    (property "Footprint" "Capacitor_THT:CP_Radial_Tantal_D5.0mm_P2.50mm" (at 136.8552 137.16 0)
+      (effects (font (size 1.27 1.27)) hide)
+    )

Commit message: changes
Connections:
- net a0: no longer U14.3
- new net A0: U14.3
Changed lines of the file:
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@@
-    (stroke (width 0) (type default))
-  )
-  (wire (pts (xy 25.4 63.5) (xy 27.94 63.5))
     (stroke (width 0) (type default))
   )
@@
   (label "d0" (at 80.01 38.1 180) (fields_autoplaced)
     (effects (font (size 1.27 1.27)) (justify right bottom))
-  )
-  (label "a0" (at 25.4 63.5 0) (fields_autoplaced)
-    (effects (font (size 1.27 1.27)) (justify left bottom))
   )
   (label "PSG1IOB0" (at 48.26 171.45 180) (fields_autoplaced)
@@
       (effects (font (size 1.27 1.27)) (justify right) hide)
     )
+  )
+  (global_label "A0" (shape input) (at 27.94 63.5 180) (fields_autoplaced)
+    (effects (font (size 1.27 1.27)) (justify right))
+    (property "Intersheetrefs" "${INTERSHEET_REFS}" (at 22.7361 63.5 0)
+      (effects (font (size 1.27 1.27)) (justify right) hide)
+    )

Commit message: layout complete for v3
Connections:
- net A0 is gone; now on net a0: U14.3
Changed lines of the file:
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@@
-    (stroke (width 0) (type default))
-  )
-  (wire (pts (xy 140.97 78.74) (xy 144.78 78.74))
     (stroke (width 0) (type default))
   )
@@
   )
   (label "PSG1IOA6" (at 102.87 69.85 0) (fields_autoplaced)
-    (effects (font (size 1.27 1.27)) (justify left bottom))
-  )
-  (label "a0" (at 140.97 78.74 0) (fields_autoplaced)
     (effects (font (size 1.27 1.27)) (justify left bottom))
   )
@@
     )
   )
+  (global_label "a0" (shape input) (at 144.78 78.74 180) (fields_autoplaced)
+    (effects (font (size 1.27 1.27)) (justify right))
+    (property "Intersheetrefs" "${INTERSHEET_REFS}" (at 139.4363 78.74 0)
+      (effects (font (size 1.27 1.27)) (justify right) hide)
+    )
+  )
   (global_label "PSG2IOA[0..7]" (shape input) (at 223.52 72.39 0) (fields_autoplaced)
     (effects (font (size 1.27 1.27)) (justify left))
@@
     )
   )
-  (global_label "A0" (shape input) (at 27.94 63.5 180) (fields_autoplaced)
-    (effects (font (size 1.27 1.27)) (justify right))
-    (property "Intersheetrefs" "${INTERSHEET_REFS}" (at 22.7361 63.5 0)
-      (effects (font (size 1.27 1.27)) (justify right) hide)
-    )
+  (global_label "a0" (shape input) (at 27.94 63.5 180) (fields_autoplaced)
+    (effects (font (size 1.27 1.27)) (justify right))
+    (property "Intersheetrefs" "${INTERSHEET_REFS}" (at 22.5963 63.5 0)
+      (effects (font (size 1.27 1.27)) (justify right) hide)
+    )

Commit message: got msbasic to work and am trying to config C
Parts:
- J19: footprint 8bits:SWITCHCRAFT_35RAPC4BV4 -> SWITCHCRAFT_35RAPC4BV4
Changed lines of the file:
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@@
       (effects (font (size 1.27 1.27)))
     )
-    (property "Footprint" "8bits:SWITCHCRAFT_35RAPC4BV4" (at 161.29 137.16 0)
+    (property "Footprint" "SWITCHCRAFT_35RAPC4BV4" (at 161.29 137.16 0)
       (effects (font (size 1.27 1.27)) (justify bottom) hide)
     )
@@
     )
   )
-  (symbol (lib_name "+5V_1") (lib_id "power:+5V") (at 238.76 30.48 0) (unit 1)
+  (symbol (lib_id "power:+5V") (at 238.76 30.48 0) (unit 1)
     (in_bom yes) (on_board yes) (dnp no) (fields_autoplaced)
     (property "Reference" "#PWR?" (at 238.76 34.29 0)
@@
     )
   )
-  (symbol (lib_name "GND_1") (lib_id "power:GND") (at 238.76 38.1 0) (unit 1)
+  (symbol (lib_id "power:GND") (at 238.76 38.1 0) (unit 1)
     (in_bom yes) (on_board yes) (dnp no) (fields_autoplaced)
     (property "Reference" "#PWR?" (at 238.76 44.45 0)
